File: circuit/murakumo/murakumo.sch (KiCad schematic (older format))
At the start: 0 parts

Commit message: hoge
Parts:
- added C? (x14): 0.1u, symbol Device:C
- added C? (x2): 2.2u, symbol Device:C
- added C?: 100n, symbol Device:C
- added C?: 1u, symbol Device:C
- added C? (x5): C, symbol Device:C
- added D?: LED, symbol Device:LED
- added D?: LED_ABGR, symbol Device:LED_ABGR
- added FB? (x2): Ferrite_Bead, symbol Device:Ferrite_Bead
- added J?: ENX_10_EASY_1, symbol Connector_Generic:Conn_02x05_Odd_Even
- added J?: SWD, symbol Connector_Generic:Conn_01x06
- added J?: MainSensor, symbol Connector_Generic:Conn_01x16
- added J?: I2C3, symbol Connector_Generic:Conn_01x04
- added J?: ENX_10_EASY_2, symbol Connector_Generic:Conn_02x05_Odd_Even
- added J?: USART1, symbol Connector_Generic:Conn_01x04
- added J?: Conn_01x04, symbol Connector_Generic:Conn_01x04
- added J?: Power, symbol Connector_Generic:Conn_01x03
- added R? (x5): R, symbol Device:R
- added R? (x4): 10k, symbol Device:R
- added SW?: RST_SW, symbol Switch:SW_MEC_5G
- added SW?: 220AMB16R, symbol Switch:SW_Coded_SH-7050
- added U?: ICM-20648, symbol ICM-20648:ICM-20648
- added U?: STM32F405RGTx, Package_QFP:LQFP-64_10x10mm_P0.5mm, symbol MCU_ST_STM32F4:STM32F405RGTx
Connections:
- net labels added: +3.3V, +5V, ADC_IN0, ADC_IN1, ADC_IN10, ADC_IN11, ADC_IN12, ADC_IN13, ADC_IN14, ADC_IN15, ADC_IN2, ADC_IN3, ADC_IN4, ADC_IN5, ADC_IN6, ADC_IN7, ADC_IN8, ADC_IN9, B, Buzzer, Cancel, DRV1_IN1, DRV1_IN2, DRV2_IN1, DRV2_IN2, ENX1_A, ENX1_B, ENX2_A, ENX2_B, Enter, G, GND, I2C3_SCL, I2C3_SDA, ICM_SCLK, ICM_SDI, ICM_SDO, ICM_nCS, LED1, LED2, R, RCC_OSC_IN, RCC_OSC_OUT, Rotary1, Rotary2, Rotary4, Rotary8, SPI2_MISO, SPI2_MOSI, SPI2_NSS, SPI2_SCK, SWCLK, SWDIO, SWO, SubSens1, SubSens2, USART1_RX, USART1_TX, VCC, VDC, VDD, VDDA, nRST
- wire segments 0 -> 184
- no-connect marks 0 -> 16

Commit message: hoge
Parts:
- removed C? (x4): 0.1u, symbol Device:C
- removed D?: LED, symbol Device:LED
- removed D?: LED_ABGR, symbol Device:LED_ABGR
- removed J?: MainSensor, symbol Connector_Generic:Conn_01x16
- removed J?: Conn_01x04, symbol Connector_Generic:Conn_01x04
- removed R? (x4): R, symbol Device:R
- removed R? (x4): 10k, symbol Device:R
- removed SW?: 220AMB16R, symbol Switch:SW_Coded_SH-7050
- added C37, C38: 0.1u, symbol Device:C
- added D1, D10, D11, D12, D2, D3, D4, D5, D6, D7, D8, D9: SIR19-21C/TR8, Diode_SMD:D_0603_1608Metric, symbol Device:LED
- added FB3: Ferrite_Bead, symbol Device:Ferrite_Bead
- added J18, J19: Conn_01x03, symbol Connector_Generic:Conn_01x03
- added J4: FrontSensor, symbol Connector_Generic:Conn_01x08
- added J7: Conn_01x05, symbol Connector_Generic:Conn_01x05
- added J9: Conn_01x11, symbol Connector_Generic:Conn_01x11
- added Q1, Q10, Q11, Q12, Q2, Q3, Q4, Q5, Q6, Q7, Q8, Q9: TEMT7100X01, TEMT7100X01:TEMT7100X01, symbol Device:Q_Photo_NPN
- added R1, R11, R13, R15, R17, R19, R21, R23, R3, R5, R7, R9: R, Resistor_SMD:R_0603_1608Metric, symbol Device:R
- added R10, R12, R14, R16, R18, R2, R20, R22, R24, R4, R6, R8: 10k, symbol Device:R
- added RN1, RN2: 10k, symbol Device:R_Pack04
- C3: renamed from C?; value 0.1u -> 4.7u
- C5: renamed from C?; value 100n -> 0.1u
- R25: renamed from R?; value R -> 10k
- SW1: renamed from SW?; value RST_SW -> RST
- gave numbers to parts that had none: 27
Connections:
- net labels added: ICM_MISO, ICM_MOSI, SW1, SW2, Sensor01, Sensor02, Sensor03, Sensor04, Sensor05, Sensor06, Sensor07, Sensor08, Sensor09, Sensor10, Sensor11, Sensor12
- net labels removed: ADC_IN0, ADC_IN1, ADC_IN10, ADC_IN11, ADC_IN12, ADC_IN13, ADC_IN14, ADC_IN15, ADC_IN2, ADC_IN3, ADC_IN4, ADC_IN5, ADC_IN6, ADC_IN7, ADC_IN8, ADC_IN9, Cancel, Enter, ICM_SDI, ICM_SDO, RCC_OSC_OUT, SPI2_MISO, SPI2_MOSI, SPI2_NSS, SPI2_SCK, VCC, VDC, VDDA
- wire segments 184 -> 384
- no-connect marks 16 -> 17
Other:
- note added: "ENCORDER"
- note added: "ForegroundSensor"
- note added: "I2C"
- note added: "InertialSensor"
- note added: "PowerSupply"
- note added: "SWD"
- note added: "SideSensor"
- note added: "USART"
- moved on the sheet: C1, C10, C11, C12, C13, C14, C15, C16, C17, C18, C19, C2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

Commit message: hoge
Parts:
- removed J18: Conn_01x03, symbol Connector_Generic:Conn_01x03
- added BZ1: TE044003-4, symbol Device:Buzzer
- added D24: RB751S40-AU_R1_000A1, symbol Device:D
- added D? (x2): LED, symbol Device:LED
- added J?: Conn_01x03, symbol Connector_Generic:Conn_01x03
- added Q17: 2N7002T, Package_TO_SOT_SMD:SOT-23, symbol Transistor_FET:2N7002
- added R31: 100, symbol Device:R
- added R32: 1k, symbol Device:R
- added R34: 36, symbol Device:R
- added R? (x2): 10k, symbol Device:R
- added R? (x2): 470, symbol Device:R
- added RN?: 10k, symbol Device:R_Pack04
- added U7: ASTMLPA-16MHz-LJ-E-T, symbol OSC:ASTMLPA-16MHz-LJ-E-T
- J9: value Conn_01x11 -> Conn_01x10; symbol Connector_Generic:Conn_01x11 -> Connector_Generic:Conn_01x10
- R1, R11, R13, R15, R17, R19, R21, R23, R3, R5, R7, R9: value R -> 100
Connections:
- net labels removed: Buzzer, RCC_OSC_IN
- wire segments 384 -> 443
- no-connect marks 17 -> 18
Other:
- note added: "20mA"
- note added: "240mA\n"
- note added: "2mA"
- note added: "36mA"
- note added: "6.2mA\n"
- note added: "90mA"
- note added: "Buzzer"
- note added: "Oscillator"
- moved on the sheet: C10, C11, C16, C17, C7, FB1, FB2, J19, J4, J7, J8, R25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

Commit message: オシレータ増やした。モータドライバの信号を CPU で読めるようにした。nRST にプルアップ抵抗を接続。まだ CPU の正しいピンに正しい線をつなげることができていない。
Parts:
- removed RN?: 10k, symbol Device:R_Pack04
- added C12: 0.1u, symbol Device:C
- added R?: 10k, symbol Device:R
- added U?: ASTMLPA-16MHz-LJ-E-T, symbol OSC:ASTMLPA-16MHz-LJ-E-T
- FB1: renamed from FB3; value Ferrite_Bead -> 470u
- FB2: renamed from FB1; value Ferrite_Bead -> 470u
- FB3: renamed from FB2; value Ferrite_Bead -> 470u
- J10: renamed from J9; value Conn_01x10 -> SWITCHandMOTORSIGNAL; symbol Connector_Generic:Conn_01x10 -> Connector_Generic:Conn_01x15
- J4: symbol Connector_Generic:Conn_01x08 -> Connector_Generic:Conn_01x06
- J6: renamed from J7; value Conn_01x05 -> LED
- R31: renamed from R32; value 1k -> 10k
- RN1: renamed from RN2; symbol Device:R_Pack04 -> Device:R_Pack03
- gave numbers to parts that had none: 7
- renumbered C37 to C1, C8 to C13, C12 to C14, C9 to C15, C15 to C16, C16 to C17, C17 to C18, C14 to C19, C38 to C2, C13 to C20, C18 to C21, C19 to C22, C1 to C3, C2 to C4, C3 to C5, C4 to C6, C5 to C7, C6 to C8, C7 to C9, D24 to D12, D10 to D13, D11 to D14, D12 to D15, J5 to J11, J19 to J2, J1 to J3, J3 to J5, J2 to J7, J6 to J8, J8 to J9, Q17 to Q10, Q10 to Q11, Q11 to Q12, Q12 to Q13, R25 to R23, R19 to R24, R20 to R25, R21 to R26, R22 to R27, R23 to R28, R24 to R29, R31 to R30, R34 to R32, RN1 to RN2, U7 to U1, U1 to U2, U2 to U3
Connections:
- net +3V3: now also J4.6 (Pin_6), RN1.4 (R3.2), C12.1, R?.1, U?.4 (Vdd); no longer J4.7 (Pin_7), J4.8 (Pin_8), RN1.7 (R2.2), RN1.8 (R1.2)
- net GND: now also U3.22 (nCS), C12.2, U?.2 (GND); no longer J4.2 (Pin_2)
- net Rotary1: now also J10.9 (Pin_9); no longer J10.5 (Pin_5)
- net Rotary2: now also J10.10 (Pin_10); no longer J10.6 (Pin_6)
- net Rotary4: now also J10.11 (Pin_11); no longer J10.7 (Pin_7)
- net Rotary8: now also J10.12 (Pin_12); no longer J10.8 (Pin_8)
- net SW1: now also J10.13 (Pin_13); no longer J10.9 (Pin_9)
- net SW2: now also J10.14 (Pin_14); no longer J10.10 (Pin_10)
- net nRST: now also R?.2
- net at U2.10 (PC2): now also J4.3 (Pin_3); no longer J4.4 (Pin_4)
- net at U2.11 (PC3): now also J4.2 (Pin_2); no longer J4.3 (Pin_3)
- net at U2.6 (PH1): now also U?.3 (OUT)
- net at U2.8 (PC0): now also J4.5 (Pin_5); no longer J4.6 (Pin_6)
- net at U2.9 (PC1): now also J4.4 (Pin_4); no longer J4.5 (Pin_5)
- net DRV1_IN1 renamed DRV1_EN
- net DRV1_EN: now also J10.3 (Pin_3); no longer J10.1 (Pin_1)
- net DRV1_IN2 renamed DRV1_PN
- net DRV1_PN: now also J10.4 (Pin_4); no longer J10.2 (Pin_2)
- net DRV2_IN1 renamed DRV2_EN
- net DRV2_EN: now also J10.7 (Pin_7); no longer J10.3 (Pin_3)
- net DRV2_IN2 renamed DRV2_PN
- net DRV2_PN: now also J10.8 (Pin_8); no longer J10.4 (Pin_4)
- removed net ICM_nCS: RN1.4 (R4.1), U2.33 (PB12), U3.22 (nCS)
- new net DRV1_nFAULT: J10.1 (Pin_1)
- new net DRV1_nSLEEP: J10.2 (Pin_2)
- new net DRV2_nFAULT: J10.5 (Pin_5)
- new net DRV2_nSLEEP: J10.6 (Pin_6)
- new net SW3: J10.15 (Pin_15), U2.33 (PB12)
Other:
- note added: "1.5mA"
- moved on the sheet: C1, C2, C3, C4, C9, D12, J6, SW1, U1

Commit message: hoge
Parts:
- removed U?: ASTMLPA-16MHz-LJ-E-T, symbol OSC:ASTMLPA-16MHz-LJ-E-T
Connections:
- net DRV1_EN: now also U2.54 (PD2); no longer U2.58 (PB6)
- net DRV1_PN: now also U2.58 (PB6); no longer U2.59 (PB7)
- net DRV1_nFAULT: now also U2.6 (PH1)
- net DRV1_nSLEEP: now also U2.2 (PC13)
- net DRV2_EN: no longer U2.61 (PB8)
- net DRV2_PN: now also U2.59 (PB7); no longer U2.62 (PB9)
- net DRV2_nFAULT: now also U2.3 (PC14)
- net DRV2_nSLEEP: now also U2.4 (PC15)
- net I2C3_SCL: no longer U2.41 (PA8)
- net I2C3_SDA: no longer U2.40 (PC9)
- net Rotary1: now also U2.45 (PA12); no longer U2.51 (PC10)
- net Rotary2: now also U2.44 (PA11); no longer U2.52 (PC11)
- net Rotary4: now also U2.43 (PA10); no longer U2.53 (PC12)
- net Rotary8: now also U2.34 (PB13); no longer U2.54 (PD2)
- net SW1: no longer U2.50 (PA15)
- net SW2: no longer U2.34 (PB13)
- net SW3: no longer U2.33 (PB12)
- net USART1_RX: no longer U2.43 (PA10)
- net USART1_TX: no longer U2.42 (PA9)
- net at R30.2: now also U2.50 (PA15); no longer U2.56 (PB4)
- net B renamed LED_B
- net LED_B: now also U2.53 (PC12); no longer U2.4 (PC15)
- net ENX1_A renamed Encorder1_A
- net Encorder1_A: now also U2.42 (PA9); no longer U2.44 (PA11)
- net ENX1_B renamed Encorder1_B
- net Encorder1_B: now also U2.41 (PA8); no longer U2.45 (PA12)
- net ENX2_A renamed Encorder2_A
- net Encorder2_A: now also U2.57 (PB5); no longer U2.37 (PC6)
- net ENX2_B renamed Encorder2_B
- net Encorder2_B: now also U2.56 (PB4); no longer U2.38 (PC7)
- net G renamed LED_G
- net LED_G: now also U2.52 (PC11); no longer U2.3 (PC14)
- net LED1 renamed LED1_White
- net LED1_White: no longer U2.57 (PB5)
- net LED2 renamed LED_Red
- net R renamed LED_R
- net LED_R: now also U2.51 (PC10); no longer U2.2 (PC13)
- new net ERV2_EN: U2.33 (PB12)
- new net I2C_SCL: U2.61 (PB8)
- new net I2C_SDA: U2.62 (PB9)
- new net LED_White1: U2.40 (PC9)
- new net USART_RX: U2.38 (PC7)
- new net USART_TX: U2.37 (PC6)
- no-connect marks 18 -> 17
Other:
- note added: "SensorBar"
- moved on the sheet: BZ1, C10, C11, C12, C13, C14, C17, C18, C19, D10, D11, D12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

Commit message: 次はフットプリントの関連付け
Parts:
- removed BZ1: TE044003-4, symbol Device:Buzzer
- removed C1, C12, C16, C17, C18, C2, C21, C22, C3, C4, C6, C7, C9: 0.1u, symbol Device:C
- removed C10, C11: 2.2u, symbol Device:C
- removed C13, C14, C15, C19, C20: C, symbol Device:C
- removed C5: 4.7u, symbol Device:C
- removed C8: 1u, symbol Device:C
- removed D1, D13, D14, D15, D2, D3, D4, D5, D6, D7, D8, D9: SIR19-21C/TR8, Diode_SMD:D_0603_1608Metric, symbol Device:LED
- removed D10, D11: LED, symbol Device:LED
- removed D12: RB751S40-AU_R1_000A1, symbol Device:D
- removed FB1, FB2, FB3: 470u, symbol Device:Ferrite_Bead
- removed J1, J2: Conn_01x03, symbol Connector_Generic:Conn_01x03
- removed J10: SWITCHandMOTORSIGNAL, symbol Connector_Generic:Conn_01x15
- removed J11: ENX_10_EASY_2, symbol Connector_Generic:Conn_02x05_Odd_Even
- removed J3: SWD, symbol Connector_Generic:Conn_01x06
- removed J4: FrontSensor, symbol Connector_Generic:Conn_01x06
- removed J5: I2C3, symbol Connector_Generic:Conn_01x04
- removed J6: LED, symbol Connector_Generic:Conn_01x05
- removed J7: ENX_10_EASY_1, symbol Connector_Generic:Conn_02x05_Odd_Even
- removed J8: USART1, symbol Connector_Generic:Conn_01x04
- removed J9: Power, symbol Connector_Generic:Conn_01x03
- removed Q1, Q11, Q12, Q13, Q2, Q3, Q4, Q5, Q6, Q7, Q8, Q9: TEMT7100X01, TEMT7100X01:TEMT7100X01, symbol Device:Q_Photo_NPN
- removed Q10: 2N7002T, Package_TO_SOT_SMD:SOT-23, symbol Transistor_FET:2N7002
- removed R1, R11, R13, R15, R17, R24, R26, R28, R3, R5, R7, R9: 100, Resistor_SMD:R_0603_1608Metric, symbol Device:R
- removed R10, R12, R14, R16, R18, R2, R21, R22, R23, R25, R27, R29, R31, R4, R6, R8, R?: 10k, symbol Device:R
- removed R19, R20: 470, symbol Device:R
- removed R30: 100, symbol Device:R
- removed R32: 36, symbol Device:R
- removed RN1: 10k, symbol Device:R_Pack03
- removed RN2: 10k, symbol Device:R_Pack04
- removed SW1: RST, symbol Switch:SW_MEC_5G
- removed U1: ASTMLPA-16MHz-LJ-E-T, symbol OSC:ASTMLPA-16MHz-LJ-E-T
- removed U2: STM32F405RGTx, Package_QFP:LQFP-64_10x10mm_P0.5mm, symbol MCU_ST_STM32F4:STM32F405RGTx
- removed U3: ICM-20648, symbol ICM-20648:ICM-20648
Connections:
- no-connect marks 17 -> 0
Other:
- note removed: "1.5mA"
- note removed: "20mA"
- note removed: "240mA\n"
- note removed: "2mA"
- note removed: "36mA"
- note removed: "6.2mA\n"
- note removed: "90mA"
- note removed: "Buzzer"
- note removed: "ENCORDER"
- note removed: "ForegroundSensor"
- note removed: "I2C"
- note removed: "InertialSensor"
- note removed: "Oscillator"
- note removed: "PowerSupply"
- note removed: "SWD"
- note removed: "SensorBar"
- note removed: "SideSensor"
- note removed: "USART"

Commit message: あとちょっとでフットプリントの関連付けが終わる
Changed lines of the file:
@@
 EELAYER 30 0
 EELAYER END
-$Descr A2 23386 16535
+$Descr A4 11693 8268
 encoding utf-8
 Sheet 1 5
@@
 $EndDescr
 $Sheet
-S 11700 8950 500  150
+S 5800 3950 500  150
 U 61E3FF76
 F0 "MurakumoFrontSens" 50
@@
 $EndSheet
 $Sheet
-S 10700 8950 500  150
+S 4800 3950 500  150
 U 61EDC519
 F0 "MurakumoPower" 50
@@
 $EndSheet
 $Sheet
-S 12700 8950 500  150
+S 6800 3950 500  150
 U 61EC4080
 F0 "MurakumoSubSens" 50
@@
 $EndSheet
 $Sheet
-S 9700 8950 500  150
+S 3800 3950 500  150
 U 624FCD7A
 F0 "Main" 50
