File: circuit/murakumo/MurakumoSens.sch (KiCad schematic (older format))
At the start: 52 parts, among them J1 Conn_01x21, Q1 TEMT7100X01, Q10 TEMT7100X01, Q11 TEMT7100X01, Q12 TEMT7100X01, Q13 TEMT7100X01, Q14 TEMT7100X01, Q15 TEMT7100X01, Q16 TEMT7100X01, Q17 TEMT7100X01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

Commit message: hoge
Parts:
- removed D17: SIR19-21C/TR8, Diode_SMD:D_0603_1608Metric, symbol Device:LED
- removed Q17: TEMT7100X01, TEMT7100X01:TEMT7100X01, symbol Device:Q_Photo_NPN
- removed R17: R, Resistor_SMD:R_0603_1608Metric, symbol Device:R
- J1: value Conn_01x21 -> Conn_01x20; symbol Connector_Generic:Conn_01x21 -> Connector_Generic:Conn_01x20
Connections:
- net labels removed: MAIN_SENSOR17
- wire segments 95 -> 90
Changed lines of the file:
@@
 	7250 4250 7250 3900
-$Comp
-L Device:Q_Photo_NPN Q17
-U 1 1 61E709C3
-P 8700 3750
-F 0 "Q17" H 8890 3796 50  0000 L CNN
-F 1 "TEMT7100X01" H 8890 3705 50  0000 L CNN
-F 2 "TEMT7100X01:TEMT7100X01" H 8900 3850 50  0001 C CNN
-F 3 "~" H 8700 3750 50  0001 C CNN
-	1    8700 3750
-	1    0    0    -1
-$EndComp
-$Comp
-L Device:LED D17
-U 1 1 61E709C9
-P 8250 3750
-F 0 "D17" V 8289 3632 50  0000 R CNN
-F 1 "SIR19-21C/TR8" V 8198 3632 50  0000 R CNN
-F 2 "Diode_SMD:D_0603_1608Metric" H 8250 3750 50  0001 C CNN
-F 3 "~" H 8250 3750 50  0001 C CNN
-	1    8250 3750
-	0    -1   -1   0
-$EndComp
-$Comp
-L power:GND #PWR054
-U 1 1 61E709CF
-P 8800 4250
-F 0 "#PWR054" H 8800 4000 50  0001 C CNN
-F 1 "GND" H 8805 4077 50  0000 C CNN
-F 2 "" H 8800 4250 50  0001 C CNN
-F 3 "" H 8800 4250 50  0001 C CNN
-	1    8800 4250
-	1    0    0    -1
-$EndComp
-Text GLabel 8800 3250 1    50   Input ~ 0
-MAIN_SENSOR17
-Wire Wire Line
-	8800 3250 8800 3550
-$Comp
-L Device:R R17
-U 1 1 61E709D7
-P 8250 3250
-F 0 "R17" H 8320 3296 50  0000 L CNN
-F 1 "R" H 8320 3205 50  0000 L CNN
-F 2 "Resistor_SMD:R_0603_1608Metric" V 8180 3250 50  0001 C CNN
-F 3 "~" H 8250 3250 50  0001 C CNN
-	1    8250 3250
-	1    0    0    -1
-$EndComp
-Wire Wire Line
-	8250 3400 8250 3600
-$Comp
-L power:+3V3 #PWR038
-U 1 1 61E709DE
-P 8250 2750
-F 0 "#PWR038" H 8250 2600 50  0001 C CNN
-F 1 "+3V3" H 8265 2923 50  0000 C CNN
-F 2 "" H 8250 2750 50  0001 C CNN
-F 3 "" H 8250 2750 50  0001 C CNN
-	1    8250 2750
-	1    0    0    -1
-$EndComp
-Wire Wire Line
-	8250 2750 8250 3100
-$Comp
-L power:GND #PWR053
-U 1 1 61E709E5
-P 8250 4250
-F 0 "#PWR053" H 8250 4000 50  0001 C CNN
-F 1 "GND" H 8255 4077 50  0000 C CNN
-F 2 "" H 8250 4250 50  0001 C CNN
-F 3 "" H 8250 4250 50  0001 C CNN
-	1    8250 4250
-	1    0    0    -1
-$EndComp
-Wire Wire Line
-	8800 4250 8800 3950
-Wire Wire Line
-	8250 4250 8250 3900
 $Comp
 L Device:Q_Photo_NPN Q10
@@
 	9750 2250 9750 1900
 Wire Wire Line
-	1250 5000 1250 4900
-Connection ~ 1250 5000
+	1250 4900 1250 4800
+Connection ~ 1250 4900
 Wire Wire Line
-	900  5000 1250 5000
+	900  4900 1250 4900
 Wire Wire Line
-	1250 4900 900  4900
+	1250 4800 900  4800
 Wire Wire Line
-	1250 5250 1250 5000
+	1250 5150 1250 4900
 $Comp
 L power:GND #PWR055
 U 1 1 61FE385E
-P 1250 5250
-F 0 "#PWR055" H 1250 5000 50  0001 C CNN
-F 1 "GND" H 1255 5077 50  0000 C CNN
-F 2 "" H 1250 5250 50  0001 C CNN
-F 3 "" H 1250 5250 50  0001 C CNN
-	1    1250 5250
+P 1250 5150
+F 0 "#PWR055" H 1250 4900 50  0001 C CNN
+F 1 "GND" H 1255 4977 50  0000 C CNN
+F 2 "" H 1250 5150 50  0001 C CNN
+F 3 "" H 1250 5150 50  0001 C CNN
+	1    1250 5150
 	1    0    0    -1
 $EndComp
@@
 	1    0    0    -1
 $EndComp
-Text GLabel 900  4800 2    50   Input ~ 0
-MAIN_SENSOR17
 Text GLabel 900  4700 2    50   Input ~ 0
 MAIN_SENSOR16
@@
 MAIN_SENSOR01
 $Comp
-L Connector_Generic:Conn_01x21 J1
+L Connector_Generic:Conn_01x20 J1
 U 1 1 61F8CE2E
 P 700 4000
 F 0 "J1" H 618 2775 50  0000 C CNN
-F 1 "Conn_01x21" H 618 2866 50  0000 C CNN
+F 1 "Conn_01x20" H 618 2866 50  0000 C CNN
 F 2 "" H 700 4000 50  0001 C CNN
 F 3 "~" H 700 4000 50  0001 C CNN
