File: circuit/murakumo/MurakumoFrontSens.sch (KiCad schematic (older format))
At the start: 14 parts, among them J10 FFC, Q13 TEMT7100X01, Q14 TEMT7100X01, Q15 TEMT7100X01, Q16 TEMT7100X01

Commit message: hoge
Parts:
- R26, R27, R28, R29: value R -> 100
Other:
- note added: "81.32mA\n"
Changed lines of the file:
@@
 AR Path="/62D533E7" Ref="R?"  Part="1"
 F 0 "R26" H 3870 4396 50  0000 L CNN
-F 1 "R" H 3870 4305 50  0000 L CNN
+F 1 "100" H 3870 4305 50  0000 L CNN
 F 2 "Resistor_SMD:R_0603_1608Metric" V 3730 4350 50  0001 C CNN
 F 3 "~" H 3800 4350 50  0001 C CNN
@@
 AR Path="/62D56ECF" Ref="R?"  Part="1"
 F 0 "R27" H 4670 4396 50  0000 L CNN
-F 1 "R" H 4670 4305 50  0000 L CNN
+F 1 "100" H 4670 4305 50  0000 L CNN
 F 2 "Resistor_SMD:R_0603_1608Metric" V 4530 4350 50  0001 C CNN
 F 3 "~" H 4600 4350 50  0001 C CNN
@@
 AR Path="/62D57F7A" Ref="R?"  Part="1"
 F 0 "R28" H 5470 4396 50  0000 L CNN
-F 1 "R" H 5470 4305 50  0000 L CNN
+F 1 "100" H 5470 4305 50  0000 L CNN
 F 2 "Resistor_SMD:R_0603_1608Metric" V 5330 4350 50  0001 C CNN
 F 3 "~" H 5400 4350 50  0001 C CNN
@@
 AR Path="/62D5EEE7" Ref="R?"  Part="1"
 F 0 "R29" H 6270 4396 50  0000 L CNN
-F 1 "R" H 6270 4305 50  0000 L CNN
+F 1 "100" H 6270 4305 50  0000 L CNN
 F 2 "Resistor_SMD:R_0603_1608Metric" V 6130 4350 50  0001 C CNN
 F 3 "~" H 6200 4350 50  0001 C CNN
@@
 Wire Wire Line
 	6900 2250 6900 2150
+Text Notes 2350 2500 0    50   ~ 0
+81.32mA\n
 $EndSCHEMATC

Commit message: オシレータ増やした。モータドライバの信号を CPU で読めるようにした。nRST にプルアップ抵抗を接続。まだ CPU の正しいピンに正しい線をつなげることができていない。
Parts:
- added R33, R34, R35, R36: 10k, symbol Device:R
- J12: renamed from J10; value FFC -> Micon; symbol Connector_Generic:Conn_01x08 -> Connector_Generic:Conn_01x06
- renumbered C20 to C23, D13 to D16, D14 to D17, D15 to D18, D16 to D19, Q13 to Q14, Q14 to Q15, Q15 to Q16, Q16 to Q17, R26 to R37, R27 to R38, R28 to R39, R29 to R40
Connections:
- net +3V3: now also J12.6 (Pin_6), R33.1, R34.1, R35.1, R36.1; no longer J12.7 (Pin_7), J12.8 (Pin_8)
- net GND: no longer J12.2 (Pin_2)
- net at Q14.1 (C): now also J12.2 (Pin_2), R33.2; no longer J12.3 (Pin_3)
- net at Q15.1 (C): now also J12.3 (Pin_3), R34.2; no longer J12.4 (Pin_4)
- net at Q16.1 (C): now also J12.4 (Pin_4), R35.2; no longer J12.5 (Pin_5)
- net at Q17.1 (C): now also J12.5 (Pin_5), R36.2; no longer J12.6 (Pin_6)
Other:
- note added: "20mA"
- note added: "Max160mA"
- note added: "Max20mA"
- note removed: "81.32mA\n"

Commit message: 次はフットプリントの関連付け
Parts:
- R1: renamed from R33; footprint (none) -> Resistor_SMD:R_0603_1608Metric
- R3: renamed from R35; footprint (none) -> Resistor_SMD:R_0603_1608Metric
- R6: renamed from R38; footprint Resistor_SMD:R_0603_1608Metric -> (none)
- R8: renamed from R40; footprint Resistor_SMD:R_0603_1608Metric -> (none)
- renumbered C23 to C1, D16 to D1, D17 to D2, D18 to D3, D19 to D4, J12 to J1, Q14 to Q1, Q15 to Q2, Q16 to Q3, Q17 to Q4, R34 to R2, R36 to R4, R37 to R5, R39 to R7

Commit message: あとちょっとでフットプリントの関連付けが終わる
Parts:
- C1: footprint (none) -> Capacitor_SMD:C_0603_1608Metric
- J1: value Micon -> FFC6; footprint (none) -> FFC:Molex_0545480671_01x06_P0.5mm
- R2, R4, R6, R8: footprint (none) -> Resistor_SMD:R_0603_1608Metric
Changed lines of the file:
@@
 F 0 "R6" H 4670 4396 50  0000 L CNN
 F 1 "100" H 4670 4305 50  0000 L CNN
-F 2 "" V 4530 4350 50  0001 C CNN
+F 2 "Resistor_SMD:R_0603_1608Metric" V 4530 4350 50  0001 C CNN
 F 3 "~" H 4600 4350 50  0001 C CNN
 	1    4600 4350
@@
 F 0 "R8" H 6270 4396 50  0000 L CNN
 F 1 "100" H 6270 4305 50  0000 L CNN
-F 2 "" V 6130 4350 50  0001 C CNN
+F 2 "Resistor_SMD:R_0603_1608Metric" V 6130 4350 50  0001 C CNN
 F 3 "~" H 6200 4350 50  0001 C CNN
 	1    6200 4350
@@
 P 3100 2450
 F 0 "J1" H 3400 2400 50  0000 C CNN
-F 1 "Micon" H 3400 2500 50  0000 C CNN
-F 2 "" H 3100 2450 50  0001 C CNN
+F 1 "FFC6" H 3400 2500 50  0000 C CNN
+F 2 "FFC:Molex_0545480671_01x06_P0.5mm" H 3100 2450 50  0001 C CNN
 F 3 "~" H 3100 2450 50  0001 C CNN
 	1    3100 2450
@@
 F 0 "C1" H 7015 2446 50  0000 L CNN
 F 1 "0.1u" H 7015 2355 50  0000 L CNN
-F 2 "" H 6938 2250 50  0001 C CNN
+F 2 "Capacitor_SMD:C_0603_1608Metric" H 6938 2250 50  0001 C CNN
 F 3 "~" H 6900 2400 50  0001 C CNN
 	1    6900 2400
@@
 F 0 "R2" H 4670 2046 50  0000 L CNN
 F 1 "10k" H 4670 1955 50  0000 L CNN
-F 2 "" V 4530 2000 50  0001 C CNN
+F 2 "Resistor_SMD:R_0603_1608Metric" V 4530 2000 50  0001 C CNN
 F 3 "~" H 4600 2000 50  0001 C CNN
 	1    4600 2000
@@
 F 0 "R4" H 6270 2046 50  0000 L CNN
 F 1 "10k" H 6270 1955 50  0000 L CNN
-F 2 "" V 6130 2000 50  0001 C CNN
+F 2 "Resistor_SMD:R_0603_1608Metric" V 6130 2000 50  0001 C CNN
 F 3 "~" H 6200 2000 50  0001 C CNN
 	1    6200 2000
