File: circuit/murakumo/MurakumoPower.sch (KiCad schematic (older format))
At the start: 21 parts

Commit message: hoge
Parts:
- removed J?: Conn_01x10, symbol Connector_Generic:Conn_01x10
- added J?: Conn_01x04, symbol Connector_Generic:Conn_01x04
Connections:
- net labels removed: D1_FAULT, D1_IPROPI, D1_SLEEP, D2_FAULT, D2_IPROPI, D2_SLEEP
- wire segments 112 -> 107
Changed lines of the file:
@@
 encoding utf-8
 Sheet 3 4
-Title "Murakumo Motor Circuit"
+Title "Murakumo Power Circuit"
 Date ""
 Rev ""
@@
 	1    0    0    -1
 $EndComp
-$Comp
-L Connector_Generic:Conn_01x10 J?
-U 1 1 61F1B58E
-P 3600 4000
-F 0 "J?" H 3518 3275 50  0000 C CNN
-F 1 "Conn_01x10" H 3518 3366 50  0000 C CNN
-F 2 "" H 3600 4000 50  0001 C CNN
-F 3 "~" H 3600 4000 50  0001 C CNN
-	1    3600 4000
-	-1   0    0    1
-$EndComp
 Wire Wire Line
 	4100 5350 5150 5350
 Entry Wire Line
-	4550 5250 4450 5150
+	4800 5250 4700 5150
 Entry Wire Line
-	4550 5150 4450 5050
+	4800 5150 4700 5050
 Entry Wire Line
-	4550 5050 4450 4950
+	4600 4300 4700 4400
 Entry Wire Line
-	4550 4950 4450 4850
-Entry Wire Line
-	4450 4950 4550 5050
-Entry Wire Line
-	4350 4000 4450 4100
-Entry Wire Line
-	4350 4100 4450 4200
-Entry Wire Line
-	4350 4200 4450 4300
-Entry Wire Line
-	4350 4300 4450 4400
-Text Label 4550 4950 0    50   ~ 0
-D1_FAULT
-Text Label 4550 5050 0    50   ~ 0
-D1_SLEEP
-Text Label 4550 5150 0    50   ~ 0
+	4600 4400 4700 4500
+Text Label 4800 5150 0    50   ~ 0
 D1_IN1
-Text Label 4550 5250 0    50   ~ 0
+Text Label 4800 5250 0    50   ~ 0
 D1_IN2
 Wire Wire Line
@@
 Wire Wire Line
 	4650 5550 5150 5550
-Entry Wire Line
-	4350 4400 4450 4500
-Wire Wire Line
-	4550 4950 5050 4950
 Connection ~ 5050 4950
-Wire Wire Line
-	4550 5050 5150 5050
-Wire Wire Line
-	4550 5150 5150 5150
-Wire Wire Line
-	4550 5250 5150 5250
-Entry Wire Line
-	4450 5450 4550 5550
-Wire Wire Line
-	4550 5550 4650 5550
-Connection ~ 4650 5550
-Text Label 4550 5550 0    50   ~ 0
-D1_IPROPI
-Text Label 3950 4000 0    50   ~ 0
-D1_FAULT
-Text Label 3950 4100 0    50   ~ 0
-D1_SLEEP
-Text Label 3950 4200 0    50   ~ 0
+Text Label 4600 4400 2    50   ~ 0
 D1_IN1
-Text Label 3950 4300 0    50   ~ 0
+Text Label 4600 4300 2    50   ~ 0
 D1_IN2
-Wire Wire Line
-	3800 4000 4350 4000
-Wire Wire Line
-	3800 4100 4350 4100
-Wire Wire Line
-	3800 4200 4350 4200
-Wire Wire Line
-	3800 4300 4350 4300
-Wire Wire Line
-	3800 4400 4350 4400
-Text Label 3950 4400 0    50   ~ 0
-D1_IPROPI
 Wire Wire Line
 	6650 5350 6650 5250
@@
 Entry Wire Line
 	8100 5150 8000 5050
-Entry Wire Line
-	8100 5050 8000 4950
-Entry Wire Line
-	8100 4950 8000 4850
-Entry Wire Line
-	8000 4950 8100 5050
-Text Label 8100 4950 0    50   ~ 0
-D2_FAULT
-Text Label 8100 5050 0    50   ~ 0
-D2_SLEEP
 Text Label 8100 5150 0    50   ~ 0
 D2_IN1
@@
 Wire Wire Line
 	8200 5550 8700 5550
-Wire Wire Line
-	8100 4950 8600 4950
 Connection ~ 8600 4950
 Wire Wire Line
-	8100 5050 8700 5050
-Wire Wire Line
 	8100 5150 8700 5150
 Wire Wire Line
 	8100 5250 8700 5250
-Entry Wire Line
-	8000 5450 8100 5550
-Wire Wire Line
-	8100 5550 8200 5550
-Connection ~ 8200 5550
-Text Label 8100 5550 0    50   ~ 0
-D2_IPROPI
 Wire Wire Line
 	10200 5350 10200 5250
@@
 $EndComp
 Entry Wire Line
-	4450 3800 4350 3900
+	4700 4100 4600 4200
 Entry Wire Line
-	4450 3700 4350 3800
-Entry Wire Line
-	4450 3600 4350 3700
-Entry Wire Line
-	4450 3500 4350 3600
-Entry Wire Line
-	4450 3400 4350 3500
-Text Label 3950 3500 0    50   ~ 0
-D2_FAULT
-Text Label 3950 3600 0    50   ~ 0
-D2_SLEEP
-Text Label 3950 3700 0    50   ~ 0
+	4700 4000 4600 4100
+Text Label 4600 4200 2    50   ~ 0
 D2_IN1
-Text Label 3950 3800 0    50   ~ 0
+Text Label 4600 4100 2    50   ~ 0
 D2_IN2
-Wire Wire Line
-	3800 3500 4350 3500
-Wire Wire Line
-	3800 3600 4350 3600
-Wire Wire Line
-	3800 3700 4350 3700
-Wire Wire Line
-	3800 3800 4350 3800
-Wire Wire Line
-	3800 3900 4350 3900
-Text Label 3950 3900 0    50   ~ 0
-D2_IPROPI
+$Comp
+L power:PWR_FLAG #FLG?
+U 1 1 61EF4312
+P 6700 7200
+F 0 "#FLG?" H 6700 7275 50  0001 C CNN
+F 1 "PWR_FLAG" H 6700 7373 50  0000 C CNN
+F 2 "" H 6700 7200 50  0001 C CNN
+F 3 "~" H 6700 7200 50  0001 C CNN
+	1    6700 7200
+	1    0    0    -1
+$EndComp
+$Comp
+L power:PWR_FLAG #FLG?
+U 1 1 61EF4D26
+P 5700 7450
+F 0 "#FLG?" H 5700 7525 50  0001 C CNN
+F 1 "PWR_FLAG" H 5700 7623 50  0000 C CNN
+F 2 "" H 5700 7450 50  0001 C CNN
+F 3 "~" H 5700 7450 50  0001 C CNN
+	1    5700 7450
+	-1   0    0    1
+$EndComp
+$Comp
+L power:PWR_FLAG #FLG?
+U 1 1 61EF5009
+P 6200 7450
+F 0 "#FLG?" H 6200 7525 50  0001 C CNN
+F 1 "PWR_FLAG" H 6200 7623 50  0000 C CNN
+F 2 "" H 6200 7450 50  0001 C CNN
+F 3 "~" H 6200 7450 50  0001 C CNN
+	1    6200 7450
+	-1   0    0    1
+$EndComp
+$Comp
+L power:+BATT #PWR?
+U 1 1 61EF545B
+P 6200 7200
+F 0 "#PWR?" H 6200 7050 50  0001 C CNN
+F 1 "+BATT" H 6215 7373 50  0000 C CNN
+F 2 "" H 6200 7200 50  0001 C CNN
+F 3 "" H 6200 7200 50  0001 C CNN
+	1    6200 7200
+	1    0    0    -1
+$EndComp
+$Comp
+L power:VCC #PWR?
+U 1 1 61EF58C4
+P 5700 7200
+F 0 "#PWR?" H 5700 7050 50  0001 C CNN
+F 1 "VCC" H 5715 7373 50  0000 C CNN
+F 2 "" H 5700 7200 50  0001 C CNN
+F 3 "" H 5700 7200 50  0001 C CNN
+	1    5700 7200
+	1    0    0    -1
+$EndComp
+$Comp
+L power:GND #PWR?
+U 1 1 61EF5D3D
+P 6700 7450
+F 0 "#PWR?" H 6700 7200 50  0001 C CNN
+F 1 "GND" H 6705 7277 50  0000 C CNN
+F 2 "" H 6700 7450 50  0001 C CNN
+F 3 "" H 6700 7450 50  0001 C CNN
+	1    6700 7450
+	1    0    0    -1
+$EndComp
+Wire Wire Line
+	6200 7200 6200 7450
+Wire Wire Line
+	5700 7450 5700 7200
+Wire Wire Line
+	6700 7450 6700 7200
+Wire Wire Line
+	5050 4950 5050 5050
+Wire Wire Line
+	5050 5050 5150 5050
+Wire Wire Line
+	8600 5050 8600 4950
+Wire Wire Line
+	8600 5050 8700 5050
+$Comp
+L Connector_Generic:Conn_01x04 J?
+U 1 1 61F6ED9A
+P 4050 4300
+F 0 "J?" H 3968 3875 50  0000 C CNN
+F 1 "Conn_01x04" H 3968 3966 50  0000 C CNN
+F 2 "" H 4050 4300 50  0001 C CNN
+F 3 "~" H 4050 4300 50  0001 C CNN
+	1    4050 4300
+	-1   0    0    1
+$EndComp
+Wire Wire Line
+	4800 5150 5150 5150
+Wire Wire Line
+	5150 5250 4800 5250
+Wire Wire Line
+	4250 4100 4600 4100
+Wire Wire Line
+	4600 4200 4250 4200
+Wire Wire Line
+	4250 4400 4600 4400
+Wire Wire Line
+	4600 4300 4250 4300
 Wire Bus Line
-	4450 2900 8000 2900
+	4700 3750 8000 3750
 Wire Bus Line
-	8000 2900 8000 5450
+	4700 3750 4700 4100
 Wire Bus Line
-	4450 2900 4450 3800
+	8000 3750 8000 5150
 Wire Bus Line
-	4450 4100 4450 5150
+	4700 4400 4700 5150
 $EndSCHEMATC

Commit message: hoge
Parts:
- added BZ1: TE044003-4, symbol Device:Buzzer
- added C21, C22, C23, C24, C25: 0.1u, symbol Device:C
- added C26: C, symbol Device:C
- added D17: LED_ABGR, symbol Device:LED_ABGR
- added D18, D19: LED, symbol Device:LED
- added J14: Conn_01x03, symbol Connector_Generic:Conn_01x03
- added J15: Conn_01x05, symbol Connector_Generic:Conn_01x05
- added Q17: 2N7000, Package_TO_SOT_THT:TO-92_Inline, symbol Transistor_FET:2N7000
- added R30, R33: 10k, symbol Device:R
- added R31: 0, symbol Device:R
- added R32, R34, R35, R44, R45, R46, R47, R48: R, symbol Device:R
- added RN3: R_Pack04, symbol Device:R_Pack04
- added SW2: 220AMB16R, symbol Switch:SW_Coded_SH-7050
- added SW3: SW1, symbol Switch:SW_MEC_5G
- added SW4: SW2, symbol Switch:SW_MEC_5G
- J11: renamed from J?; value Conn_01x04 -> Conn_01x11; symbol Connector_Generic:Conn_01x04 -> Connector_Generic:Conn_01x11
- gave numbers to parts that had none: 20
Connections:
- net labels added: +3.3V, +5V, Rotary1, Rotary2, Rotary4, Rotary8
- net labels removed: D1_IN1, D1_IN2
- wire segments 107 -> 216
Other:
- moved on the sheet: C27, C28, C29, C30, C31, C32, C33, C34, J12, J13, R36, R37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

Commit message: hoge
Parts:
- removed BZ1: TE044003-4, symbol Device:Buzzer
- removed Q17: 2N7000, Package_TO_SOT_THT:TO-92_Inline, symbol Transistor_FET:2N7000
- removed R31: 0, symbol Device:R
- removed R32, R34, R35: R, symbol Device:R
- added J20: Conn_01x02, symbol Connector_Generic:Conn_01x02
- D18: value LED -> White
- D19: value LED -> Red
- J11: value Conn_01x11 -> Conn_01x10; symbol Connector_Generic:Conn_01x11 -> Connector_Generic:Conn_01x10
- R38: value Rref1 -> 16k
- R40, R41: value Rref2 -> 50k
- R42, R43: value Ripropi -> 1.2k
- R44: value R -> 82
- R45, R46: value R -> 680
- R47, R48: value R -> 330
- RN3: value R_Pack04 -> 10k
- renumbered R39 to 16k1
Connections:
- net labels removed: VCC
- wire segments 216 -> 199
Other:
- note added: "1.32mA\n"
- note added: "13mA"
- note added: "330uA"
- note added: "330uA\n"
- note added: "50uA"
- note added: "LED"
- note added: "Switch"

Commit message: オシレータ増やした。モータドライバの信号を CPU で読めるようにした。nRST にプルアップ抵抗を接続。まだ CPU の正しいピンに正しい線をつなげることができていない。
Parts:
- removed 16k1: Rref1, symbol Device:R
- added C24, C26, C29, C30: 10u, symbol Device:CP
- added C25, C27, C28, C36: 0.1u, symbol Device:C
- added D20: D_Schottky, symbol Device:D_Schottky
- added Q18: CXDM4060P, symbol Device:Q_PMOS_GDS
- added R41, R43: 10k, symbol Device:R
- added R48: 16k, symbol Device:R
- added SW2: SW_DPDT_x2, symbol Switch:SW_DPDT_x2
- added SW5: SW2, symbol Switch:SW_MEC_5G
- added U4: NCV7805BD2TG, symbol Regulator:Regulator_IGO
- added U5: LT1963EST-3.3#PBF, symbol Regulator:LT1963EST-3.3#PBF
- J14: renamed from J11; value Conn_01x10 -> CPU_GPIOandTIMER; symbol Connector_Generic:Conn_01x10 -> Connector_Generic:Conn_01x15
- J15: renamed from J12; value Conn_01x02 -> Motor
- J16: renamed from J13; value Conn_01x02 -> Motor
- J17: renamed from J14; value Conn_01x03 -> Power
- J18: renamed from J15; value Conn_01x05 -> CPU_GPIO
- SW4: value SW2 -> SW3
- renumbered C22 to C31, C23 to C32, C24 to C33, C25 to C34, C26 to C35, C21 to C37, C27 to C38, C28 to C39, C29 to C40, C30 to C41, C31 to C42, C32 to C43, C33 to C44, C34 to C45, D17 to D21, D18 to D22, D19 to D23, J20 to J13, R33 to R42, R30 to R44, R36 to R45, R37 to R46, R38 to R47, R40 to R49, R41 to R50, R42 to R51, R43 to R52, R44 to R53, R45 to R54, R46 to R55, R47 to R56, R48 to R57, SW2 to SW3, SW3 to SW6, U3 to U6, U4 to U7
Connections:
- net labels added: DRV1_EN, DRV1_PN, DRV1_nFAULT, DRV1_nSLEEP, DRV2_EN, DRV2_PN, DRV2_nFAULT, DRV2_nSLEEP, DRV2_uSLEEP, SW1, SW2, SW3
- net labels removed: D2_IN1, D2_IN2
- wire segments 199 -> 274
- no-connect marks 0 -> 1
Other:
- note added: "2mA"
- note added: "5mA"
- note added: "Driver"
- note added: "Power"
- note added: "RotarySwitch"
- note removed: "13mA"
- moved on the sheet: C31, C32, C33, C34, C35, C37, J13, J17, R42, R44, R47, R49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

Commit message: hoge
Parts:
- added J?: CPU_TIMER, symbol Connector_Generic:Conn_01x08
- J14: value CPU_GPIOandTIMER -> CPU_GPIO; symbol Connector_Generic:Conn_01x15 -> Connector_Generic:Conn_01x07
Connections:
- net DRV1_EN: now also J?.3 (Pin_3); no longer J14.3 (Pin_3)
- net DRV1_PN: now also J?.4 (Pin_4); no longer J14.4 (Pin_4)
- net DRV1_nFAULT: now also J?.1 (Pin_1); no longer J14.1 (Pin_1)
- net DRV1_nSLEEP: now also J?.2 (Pin_2); no longer J14.2 (Pin_2)
- net DRV2_EN: now also J?.7 (Pin_7); no longer J14.7 (Pin_7)
- net DRV2_PN: now also J?.8 (Pin_8); no longer J14.8 (Pin_8)
- net DRV2_nFAULT: now also J?.5 (Pin_5); no longer J14.5 (Pin_5)
- net DRV2_uSLEEP: now also J?.6 (Pin_6); no longer J14.6 (Pin_6)
- net Rotary1: now also J14.1 (Pin_1); no longer J14.9 (Pin_9)
- net Rotary2: now also J14.2 (Pin_2); no longer J14.10 (Pin_10)
- net Rotary4: now also J14.3 (Pin_3); no longer J14.11 (Pin_11)
- net Rotary8: now also J14.4 (Pin_4); no longer J14.12 (Pin_12)
- net SW1: now also J14.5 (Pin_5); no longer J14.13 (Pin_13)
- net SW2: now also J14.6 (Pin_6); no longer J14.14 (Pin_14)
- net SW3: now also J14.7 (Pin_7); no longer J14.15 (Pin_15)
Other:
- moved on the sheet: C35, C36, C37, R42, R43, R44, SW4, SW5, SW6

Commit message: 次はフットプリントの関連付け
Parts:
- removed C24: 10u, symbol Device:CP
- removed C25, C27, C28: 0.1u, symbol Device:C
- removed D20: D_Schottky, symbol Device:D_Schottky
- removed U5: LT1963EST-3.3#PBF, symbol Regulator:LT1963EST-3.3#PBF
- added C3: 22u, symbol Device:CP
- added C6: 220u, symbol Device:CP
- added C7: 0.1u, symbol Device:C
- added D10: SMLEN3WBC8W1, Diode_SMD:D_0603_1608Metric, symbol Device:LED
- added D5: SS2040FL-AU_R1_000A1, Diode_SMD:D_0603_1608Metric, symbol Device:D
- added D6: Red, Diode_SMD:D_0603_1608Metric, symbol Device:LED
- added D7: Orange, Diode_SMD:D_0603_1608Metric, symbol Device:LED
- added D8: Yellow, Diode_SMD:D_0603_1608Metric, symbol Device:LED
- added FB1: 470, symbol Device:Ferrite_Bead
- added R10: 2k, symbol Device:R
- added R11: 680, Resistor_SMD:R_0603_1608Metric, symbol Device:R
- added R12: 270, symbol Device:R
- added R19: 470, symbol Device:R
- added U2: AZ1117IH-3.3TRG1, Package_QFP:LQFP-64_10x10mm_P0.5mm, symbol Regulator:Regulator_GOI
- C12: renamed from C35; value C -> 0.1u
- C5: renamed from C30; value 10u -> 22u
- D11: renamed from D22; value White -> SMLEN3WBC8W1; footprint (none) -> original:SOD-523
- D12: renamed from D23; value Red -> SML31UT; footprint (none) -> Diode_SMD:D_0603_1608Metric
- D9: renamed from D21; value LED_ABGR -> APTF1616LSEEZGKQBKC; footprint (none) -> Diode_SMD:D_0603_1608Metric
- J5: renamed from J?; symbol Connector_Generic:Conn_01x08 -> Connector_Generic:Conn_01x04
- J8: renamed from J18; symbol Connector_Generic:Conn_01x05 -> Connector_Generic:Conn_01x06
- Q5: renamed from Q18; footprint (none) -> TEMT7100X01:TEMT7100X01
- R14: renamed from R43; footprint (none) -> Resistor_SMD:R_0603_1608Metric
- R16: renamed from R45; footprint (none) -> Resistor_SMD:R_0603_1608Metric
- R18: renamed from R48; footprint (none) -> Resistor_SMD:R_0603_1608Metric
- R20: renamed from R53; value 82 -> 470
- R21: renamed from R54; value 680 -> 1.5k
- R25: renamed from R52; footprint (none) -> Resistor_SMD:R_0603_1608Metric
- R26: renamed from R55; value 680 -> 1.5k
- R27: renamed from R56; value 330 -> 1.2k; footprint (none) -> Resistor_SMD:R_0603_1608Metric
- R28: renamed from R57; value 330 -> 1.2k
- R29: renamed from R49; footprint (none) -> Resistor_SMD:R_0603_1608Metric
- R9: renamed from R41; footprint (none) -> Resistor_SMD:R_0603_1608Metric
- U1: renamed from U4; value NCV7805BD2TG -> AZ1117R-5.0TRE1; symbol Regulator:Regulator_IGO -> Regulator:Regulator_GOI
- U3: renamed from U6; footprint original:TSSOP_16-Pin -> (none)
- U4: renamed from U7; footprint original:TSSOP_16-Pin -> (none)
- renumbered C33 to C10, C34 to C11, C36 to C13, C37 to C14, C38 to C15, C39 to C16, C40 to C17, C41 to C18, C42 to C19, C26 to C2, C43 to C20, C44 to C21, C45 to C22, C29 to C4, C31 to C8, C32 to C9, J13 to J2, J17 to J3, J14 to J4, J15 to J6, J16 to J7, R42 to R13, R44 to R15, R46 to R17, R47 to R22, R50 to R23, R51 to R24, RN3 to RN1, SW2 to SW1, SW3 to SW2, SW4 to SW3, SW5 to SW4, SW6 to SW5
Connections:
- net DRV2_nSLEEP is gone; now on an unnamed net: U4.3 (nSLEEP)
- net +3V3: now also R12.1, U2.2 (Output); no longer D9.1 (A), R20.1, R21.1
- net +5V: now also D9.1 (A), R20.1, R21.1, U1.2 (Output), C3.1, R11.1, R19.1, U2.3 (Input); no longer U1.3 (Output)
- net +BATT: now also C6.1, C7.1, D5.2 (A), R10.1
- net DRV1_EN: now also J5.1 (Pin_1); no longer J5.3 (Pin_3)
- net DRV1_PN: now also J5.2 (Pin_2); no longer J5.4 (Pin_4)
- net DRV2_EN: now also J5.3 (Pin_3); no longer J5.7 (Pin_7)
- net DRV2_PN: now also J5.4 (Pin_4); no longer J5.8 (Pin_8)
- net GND: now also SW1.2 (B), U1.1 (GND), C3.2, C6.2, C7.2, D6.1 (K), D7.1 (K), D8.1 (K), U2.1 (GND); no longer SW1.1 (A), U1.2 (GND)
- net at C2.1: now also U1.3 (Input), FB1.1; no longer U1.1 (Input)
- net at Q5.1 (G), R9.2: now also SW1.3 (C); no longer SW1.2 (B)
- net at R26.2: now also J8.6 (Pin_6); no longer J8.5 (Pin_5)
- net at R27.2: now also J8.5 (Pin_5); no longer J8.4 (Pin_4)
- net at R28.2: now also J8.4 (Pin_4); no longer J8.3 (Pin_3)
- net DRV1_nFAULT: no longer names the net of R16.2, U3.4 (nFAULT)
- net DRV1_nFAULT: now also U3.3 (nSLEEP); no longer J5.1 (Pin_1)
- removed net DRV1_nSLEEP: J5.2 (Pin_2), U3.3 (nSLEEP)
- net DRV2_nFAULT: no longer names the net of R17.2, U4.4 (nFAULT)
- net DRV2_nFAULT: no longer J5.5 (Pin_5)
- removed net DRV2_uSLEEP: J5.6 (Pin_6)
- new net: D5.1 (K), FB1.2
- new net: D10.1 (K), J8.3 (Pin_3)
- new net: D10.2 (A), R19.2
- new net: D6.2 (A), R10.2
- new net: D7.2 (A), R11.2
- new net: D8.2 (A), R12.2
Other:
- note added: "2mA\n"
- moved on the sheet: C2, C4, C5, D11, D12, D9, J2, J3, Q5, R20, R21, R22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

Commit message: あとちょっとでフットプリントの関連付けが終わる
Parts:
- C10, C11, C12, C13, C14, C15, C17, C19, C20, C21, C22, C7, C8, C9: footprint (none) -> Capacitor_SMD:C_0603_1608Metric
- D11: footprint original:SOD-523 -> Diode_SMD:D_0603_1608Metric
- D5: footprint Diode_SMD:D_0603_1608Metric -> original:SOD-123FL
- D9: footprint Diode_SMD:D_0603_1608Metric -> original:APTF1616LSEEZGKQBKC
- FB1: footprint (none) -> Inductor_SMD:L_0603_1608Metric
- J2: value Conn_01x02 -> ILG2
- J3: value Power -> PA3
- J4: value CPU_GPIO -> FFC7; footprint (none) -> FFC:Molex_0545480771_01x07_P0.5mm
- J5: value CPU_TIMER -> FFC4; footprint (none) -> Connector_FFC-FPC:Molex_200528-0040_1x04-1MP_P1.00mm_Horizontal
- J6, J7: value Motor -> PA2
- J8: value CPU_GPIO -> FFC6; footprint (none) -> FFC:Molex_0545480671_01x06_P0.5mm
- Q5: footprint TEMT7100X01:TEMT7100X01 -> original:SOT-89
- R10: footprint (none) -> Diode_SMD:D_0603_1608Metric
- R12, R13, R15, R17, R19, R20, R21, R22, R23, R24, R26, R28: footprint (none) -> Resistor_SMD:R_0603_1608Metric
- RN1: footprint (none) -> Package_SO:SOIC-8_3.9x4.9mm_P1.27mm
- SW1: footprint (none) -> Switch:SSAJ120100
- SW2: footprint (none) -> Switch:220AMB16R
- U1: footprint (none) -> Package_TO_SOT_SMD:SOT-89-3
- U2: footprint Package_QFP:LQFP-64_10x10mm_P0.5mm -> Package_TO_SOT_SMD:SOT-223-3_TabPin2
- U3, U4: footprint (none) -> original:TSSOP_16-Pin

Commit message: 回路図とフットプリントの関連付けが終わった
Parts:
- removed D12: SML31UT, Diode_SMD:D_0603_1608Metric, symbol Device:LED
- removed R21: 1.5k, Resistor_SMD:R_0603_1608Metric, symbol Device:R
- removed SW3: SW3, symbol Switch:SW_MEC_5G
- removed SW4: SW2, symbol Switch:SW_MEC_5G
- removed SW5: SW1, symbol Switch:SW_MEC_5G
- added SW3, SW4, SW5: SKRPABE010, SKRPABE010:SKRPABE010, symbol SKRPABE010:Switch
- C16, C18: footprint (none) -> Capacitor:ECASD91B107M012K00
- C2, C4: footprint (none) -> Capacitor:AVE106M16A12T-F
- C3, C5: footprint (none) -> Capacitor:865090168010
- C6: footprint (none) -> Capacitor:EEE-1AA221XP; Spice_Model (none) -> 220u; Spice_Netlist_Enabled (none) -> Y; Spice_Primitive (none) -> C
- J2: footprint (none) -> ILG:ILG_01x02
- J3: footprint (none) -> PA:PA_01x03
- J6, J7: footprint (none) -> PA:PA_01x02
- J8: value FFC6 -> FFC5; footprint FFC:Molex_0545480671_01x06_P0.5mm -> FFC:Molex_0545480571_01x05_P0.5mm; symbol Connector_Generic:Conn_01x06 -> Connector_Generic:Conn_01x05
- renumbered R22 to R21, R23 to R22, R24 to R23, R25 to R24, R26 to R25, R27 to R26, R28 to R27, R29 to R28
Connections:
- net GND: now also SW3.2, SW4.2, SW5.2
- net SW1: now also SW5.1
- net SW2: now also SW4.1
- net SW3: now also SW3.1
- net at R25.2: now also J8.5 (Pin_5); no longer J8.6 (Pin_6)
- net at R26.2: now also J8.4 (Pin_4); no longer J8.5 (Pin_5)
- net at R27.2: now also J8.3 (Pin_3); no longer J8.4 (Pin_4)
- net at J8.1 (Pin_1): now also D11.1 (K)
- net at J8.2 (Pin_2): now also D10.1 (K); no longer D11.1 (K)
