File: circuit/murakumo/main.sch (KiCad schematic (older format))
At the start: 105 parts, among them J11 SubSens2, J12 SubSens1, J13 FrontSensor, J14 SWD, J15 LED, J16 ENX_10_EASY_1, J17 I2C, J18 Motor, J19 ENX_10_EASY_2, J20 Power, J21 Switch, J22 USART, Q10 TEMT7100X01, Q11 TEMT7100X01, Q12 TEMT7100X01, Q13 TEMT7100X01, Q14 TEMT7100X01, Q15 2N7002T, Q16 TEMT7100X01, Q17 TEMT7100X01, Q18 TEMT7100X01, Q6 TEMT7100X01, Q7 TEMT7100X01, Q8 TEMT7100X01, Q9 TEMT7100X01, SW6 RST, U7 ASTMLPA-16MHz-LJ-E-T, U8 STM32F405RGTx, U9 ICM-20648

Commit message: あとちょっとでフットプリントの関連付けが終わる
Parts:
- BZ1: footprint (none) -> Buzzer:TE044003-4
- C25, C26, C27, C28, C29, C30, C31, C32, C33, C34, C35, C36, C37, C38, C39, C40, C41, C42, C43, C44, C45, C46: footprint (none) -> Capacitor_SMD:C_0603_1608Metric
- D20, D21, D22, D23, D24: footprint (none) -> Diode_SMD:D_0603_1608Metric
- D25: footprint Diode_SMD:D_0603_1608Metric -> original:SOD-523
- FB2, FB3, FB4: footprint (none) -> Inductor_SMD:L_0603_1608Metric
- J11: value SubSens2 -> SH3
- J12: value SubSens1 -> SH3
- J13: value FrontSensor -> FFC6; footprint (none) -> FFC:Molex_0545480671_01x06_P0.5mm
- J14: value SWD -> SH6
- J15: value LED -> FFC6; footprint (none) -> FFC:Molex_0545480671_01x06_P0.5mm
- J16: value ENX_10_EASY_1 -> FTSH2x5
- J17: value I2C -> SH4
- J18: value Motor -> FFC4; footprint (none) -> Connector_FFC-FPC:Molex_200528-0040_1x04-1MP_P1.00mm_Horizontal
- J19: value ENX_10_EASY_2 -> FTSH2x5
- J20: value Power -> PA3
- J21: value Switch -> FFC7; footprint (none) -> FFC:Molex_0545480771_01x07_P0.5mm
- J22: value USART -> SH4
- Q10: footprint Package_TO_SOT_SMD:SOT-23 -> TEMT7100X01:TEMT7100X01
- Q15: footprint TEMT7100X01:TEMT7100X01 -> Package_TO_SOT_SMD:SOT-523
- Q18: footprint (none) -> TEMT7100X01:TEMT7100X01
- R32, R33, R34, R35, R36, R37, R42, R43, R44, R45, R46, R47, R48, R49, R50, R51, R52, R53, R54, R55, R56, R57, R58, R59, R60, R61, R62, R63, R64: footprint (none) -> Resistor_SMD:R_0603_1608Metric
- RN2, RN3: footprint (none) -> Package_SO:SOIC-8_3.9x4.9mm_P1.27mm
- U7: footprint original:TSSOP_16-Pin -> osc:ASTMLPA-16.000MHz-LJ-E-T
- U8: footprint (none) -> Package_QFP:LQFP-64_10x10mm_P0.5mm
- U9: footprint (none) -> ICM-20648:QFN40P300X300X95-24N

Commit message: 回路図とフットプリントの関連付けが終わった
Parts:
- removed SW6: RST, symbol Switch:SW_MEC_5G
- added SW6: SKRPABE010, SKRPABE010:SKRPABE010, symbol SKRPABE010:Switch
- J11, J12: footprint (none) -> SH:SH_01x03
- J14: footprint (none) -> SH:SH_01x06
- J15: renamed from J16; footprint (none) -> FTSH:SAMTEC_FTSH-105-01-L-D-K
- J16: renamed from J15; value FFC6 -> FFC5; footprint FFC:Molex_0545480671_01x06_P0.5mm -> FFC:Molex_0545480571_01x05_P0.5mm; symbol Connector_Generic:Conn_01x06 -> Connector_Generic:Conn_01x05
- J17, J22: footprint (none) -> SH:SH_01x04
- J19: footprint (none) -> FTSH:SAMTEC_FTSH-105-01-L-D-K
- J20: footprint (none) -> PA:PA_01x03
- RN2: symbol Device:R_Pack03 -> Device:R_Pack04
- renumbered C30 to C29, C31 to C30, C32 to C31, C33 to C32, C29 to C33, D15 to D14, D16 to D15, D17 to D16, D18 to D17, D19 to D18, D20 to D19, D21 to D20, D22 to D21, D23 to D22, D24 to D23, D25 to D24, D26 to D25, D27 to D26, D28 to D27, D29 to D28, R32 to R31, R33 to R32, R34 to R33, R35 to R34, R36 to R35, R37 to R36, R38 to R37, R39 to R38, R40 to R39, R41 to R40, R42 to R41, R43 to R42, R44 to R43, R45 to R44, R46 to R45, R47 to R46, R48 to R47, R49 to R48, R50 to R49, R51 to R50, R52 to R51, R53 to R52, R54 to R53, R55 to R54, R56 to R55, R57 to R56, R58 to R57, R59 to R58, R60 to R59, R61 to R60, R62 to R61, R63 to R62, R64 to R63
Connections:
- net +3V3: now also RN2.7 (R2.2), RN2.8 (R1.2); no longer RN2.4 (R3.2)
- net GND: now also SW6.2; no longer U9.22 (nCS)
- net LED_B: now also J16.3 (Pin_3), U8.53 (PC12); no longer J16.4 (Pin_4), U8.2 (PC13)
- net LED_G: now also J16.4 (Pin_4), U8.52 (PC11); no longer J16.5 (Pin_5), U8.53 (PC12)
- net LED_R: now also J16.5 (Pin_5), U8.51 (PC10); no longer J16.6 (Pin_6), U8.52 (PC11)
- net SW3: now also U8.2 (PC13); no longer U8.33 (PB12)
- net nRST: now also U8.7 (NRST), SW6.1
- net LED_White1 renamed LED_White
- removed net LED_White2: J16.3 (Pin_3), U8.51 (PC10)
- new net ICM_nCS: RN2.4 (R4.1), U8.33 (PB12), U9.22 (nCS)
Other:
- moved on the sheet: C33, R43
