File: circuit/murakumo/murakumo.kicad_pcb (KiCad board)
At the start: 2 copper layers, 44 parts, among them Q15 2N7002T, U3 DRV8874, U4 DRV8874, U8 STM32F405RGTx

Commit message: 回路図とフットプリントの関連付けが終わった
Parts:
- removed D1, D13, D14, D15, D16, D17, D18, D19, D2, D20, D21, D22, D23, D27, D28, D29, D3, D4: SIR19-21C/TR8, Diode_SMD:D_0603_1608Metric
- removed D10, D11, D24, D26: SMLEN3WBC8W1, Diode_SMD:D_0603_1608Metric
- removed D12: SML31UT, Diode_SMD:D_0603_1608Metric
- removed D25: RB751S40-AU_R1_000A1, original:SOD-523
- removed Q15: 2N7002T, Package_TO_SOT_SMD:SOT-23
- removed R32, R34, R36, R38, R40, R42, R45, R47, R49, R5, R56, R58, R6, R60, R7, R8: 100, Resistor_SMD:R_0603_1608Metric
- removed U3, U4: DRV8874, original:TSSOP_16-Pin
- removed U8: STM32F405RGTx, Package_QFP:LQFP-64_10x10mm_P0.5mm
