File: circuit/kicad/_autosave-Main.kicad_pcb (KiCad board)
At the start: 2 copper layers, 110.8 x 117 mm, 104 parts, among them J1 SH3, J10 PA3, J11 SH4, J2 SH3, J3 FFC6, J4 SH6, J5 FTSH2x5, J6 FFC4, J7 SH4, J8 FFC12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

Commit message: 点検
Parts:
- moved J10 0.10 mm to (-22.0, -1.40)
Routing:
- net GND: vias 156 -> 157
Changed lines of the file:
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@@
   (general
     (thickness 1.6)
-    (drawings 66)
-    (tracks 1312)
+    (drawings 70)
+    (tracks 1313)
     (zones 0)
     (modules 104)
@@
   )
   (module PA:PA_01x03 (layer F.Cu)
-    (at -22 -1.5 180)
+    (at -22 -1.4 180)
     (fp_text reference J10 (at 0 -3.533328) (layer F.SilkS)
       (effects (font (size 1 1) (thickness 0.15)))
@@
       (effects (font (size 1 1) (thickness 0.15)))
     )
-    (fp_line (start -4 -2.65) (end -4 2.65) (layer F.SilkS) (width 0.12))
-    (fp_line (start 4 -2.65) (end -4 -2.65) (layer F.SilkS) (width 0.12))
-    (fp_line (start 4 2.65) (end 4 -2.65) (layer F.SilkS) (width 0.12))
-    (fp_line (start -2.75 1.545831) (end -2.75 2.649996) (layer F.SilkS) (width 0.12))
-    (fp_line (start 2.75 1.545831) (end -2.75 1.545831) (layer F.SilkS) (width 0.12))
-    (fp_line (start -2.75 2.649996) (end -4 2.649996) (layer F.SilkS) (width 0.12))
-    (fp_line (start 4 2.649996) (end 2.75 2.649996) (layer F.SilkS) (width 0.12))
     (fp_line (start 2.75 2.649996) (end 2.75 1.545831) (layer F.SilkS) (width 0.12))
-    (pad 1 thru_hole circle (at 2.5 0 180) (size 1.2 1.2) (drill 0.7) (layers *.Cu *.Mask)
-      (net 26 "Net-(FB2-Pad1)"))
-    (pad 2 thru_hole circle (at 0 0 180) (size 1.2 1.2) (drill 0.7) (layers *.Cu *.Mask)
-      (net 27 "Net-(FB3-Pad1)"))
+    (fp_line (start 4 2.649996) (end 2.75 2.649996) (layer F.SilkS) (width 0.12))
+    (fp_line (start -2.75 2.649996) (end -4 2.649996) (layer F.SilkS) (width 0.12))
+    (fp_line (start 2.75 1.545831) (end -2.75 1.545831) (layer F.SilkS) (width 0.12))
+    (fp_line (start -2.75 1.545831) (end -2.75 2.649996) (layer F.SilkS) (width 0.12))
+    (fp_line (start 4 2.65) (end 4 -2.65) (layer F.SilkS) (width 0.12))
+    (fp_line (start 4 -2.65) (end -4 -2.65) (layer F.SilkS) (width 0.12))
+    (fp_line (start -4 -2.65) (end -4 2.65) (layer F.SilkS) (width 0.12))
     (pad 3 thru_hole circle (at -2.5 0 180) (size 1.2 1.2) (drill 0.7) (layers *.Cu *.Mask)
       (net 3 GND))
+    (pad 2 thru_hole circle (at 0 0 180) (size 1.2 1.2) (drill 0.7) (layers *.Cu *.Mask)
+      (net 27 "Net-(FB3-Pad1)"))
+    (pad 1 thru_hole circle (at 2.5 0 180) (size 1.2 1.2) (drill 0.7) (layers *.Cu *.Mask)
+      (net 26 "Net-(FB2-Pad1)"))
   )
   (module SH:SH_01x04 (layer F.Cu)
@@
       (net 1 +3V3))
   )
+  (dimension 15.4 (width 0.15) (layer Dwgs.User)
+    (gr_text "15.400 mm" (at -49.4 25.7 270) (layer Dwgs.User)
+      (effects (font (size 1 1) (thickness 0.15)))
+    )
+    (feature1 (pts (xy -26 33.4) (xy -48.686421 33.4)))
+    (feature2 (pts (xy -26 18) (xy -48.686421 18)))
+    (crossbar (pts (xy -48.1 18) (xy -48.1 33.4)))
+    (arrow1a (pts (xy -48.1 33.4) (xy -48.686421 32.273496)))
+    (arrow1b (pts (xy -48.1 33.4) (xy -47.513579 32.273496)))
+    (arrow2a (pts (xy -48.1 18) (xy -48.686421 19.126504)))
+    (arrow2b (pts (xy -48.1 18) (xy -47.513579 19.126504)))
+  )
+  (gr_line (start -41.1 33.4) (end 41.1 33.4) (layer Dwgs.User) (width 0.15))
+  (dimension 54.8 (width 0.15) (layer Dwgs.User)
+    (gr_text "54.800 mm" (at -45.30436 6 270) (layer Dwgs.User)
+      (effects (font (size 1 1) (thickness 0.15)))
+    )
+    (feature1 (pts (xy -41.1 33.4) (xy -44.590781 33.4)))
+    (feature2 (pts (xy -41.1 -21.4) (xy -44.590781 -21.4)))
+    (crossbar (pts (xy -44.00436 -21.4) (xy -44.00436 33.4)))
+    (arrow1a (pts (xy -44.00436 33.4) (xy -44.590781 32.273496)))
+    (arrow1b (pts (xy -44.00436 33.4) (xy -43.417939 32.273496)))
+    (arrow2a (pts (xy -44.00436 -21.4) (xy -44.590781 -20.273496)))
+    (arrow2b (pts (xy -44.00436 -21.4) (xy -43.417939 -20.273496)))
+  )
+  (gr_line (start -41.1 -21.4) (end 41.2 -21.4) (layer Dwgs.User) (width 0.15))
   (gr_line (start -55.416604 -23) (end -40.9 -23) (layer Edge.Cuts) (width 0.2))
   (gr_line (start -9.5 -35.5) (end -9.5 -40.5) (layer Dwgs.User) (width 0.15))
@@
   (via (at -23.6 -5.6) (size 0.7) (drill 0.3) (layers F.Cu B.Cu) (net 3))
   (via (at -32.2 -4.7) (size 0.7) (drill 0.3) (layers F.Cu B.Cu) (net 3))
+  (via (at 26.6 2.8) (size 0.7) (drill 0.3) (layers F.Cu B.Cu) (net 3))
   (segment (start 17.875 -5.25) (end 20 -5.25) (width 0.25) (layer F.Cu) (net 4))
   (segment (start 20.75 -6) (end 20.75 -7.975) (width 0.25) (layer F.Cu) (net 4))
@@
     (connect_pads (clearance 0.508))
     (min_thickness 0.254)
-    (fill yes (arc_segments 32) (thermal_gap 0.508) (thermal_bridge_width 0.508))
+    (fill (arc_segments 32) (thermal_gap 0.508) (thermal_bridge_width 0.508))
     (polygon
       (pts
@@
     (connect_pads (clearance 0.508))
     (min_thickness 0.254)
-    (fill yes (arc_segments 32) (thermal_gap 0.508) (thermal_bridge_width 0.508))
+    (fill (arc_segments 32) (thermal_gap 0.508) (thermal_bridge_width 0.508))
     (polygon
       (pts
@@
       )
     )
+  )
+  (zone (net 0) (net_name "") (layers F&B.Cu) (hatch edge 0.508)
+    (connect_pads (clearance 0.508))
+    (min_thickness 0.254)
+    (keepout (tracks allowed) (vias allowed) (copperpour not_allowed))
+    (fill (arc_segments 32) (thermal_gap 0.508) (thermal_bridge_width 0.508))
+    (polygon
+      (pts
+        (xy 14.1 11.5) (xy 7.1 11.5) (xy 7.1 4.5)
+      )
+    )
