File: circuit/kicad/_autosave-Power.kicad_pcb (KiCad board)
At the start: 2 copper layers, 78.8 x 54.8 mm, 66 parts, among them J1 ILG2, J2 PA3, J3 FFC4, J4 FFC7, J5 PA2, J6 PA2, Q1 CXDM4060P, SW1 SW_DPDT_x2, SW2 220AMB16R, SW3 SKRPABE010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

Commit message: 点検
Routing:
- net +5V: track 51.7 -> 84.2 mm, vias 1 -> 2
- net +3V3: track 82.8 -> 104.1 mm
- net GND: vias 68 -> 65
Changed lines of the file:
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@@
   (general
     (thickness 1.6)
-    (drawings 24)
-    (tracks 496)
+    (drawings 23)
+    (tracks 504)
     (zones 0)
     (modules 66)
@@
   (page A4)
   (layers
-    (0 F.Cu signal hide)
-    (31 B.Cu signal hide)
+    (0 F.Cu signal)
+    (31 B.Cu signal)
     (32 B.Adhes user)
     (33 F.Adhes user)
@@
   )
   (setup
-    (last_trace_width 2.46)
+    (last_trace_width 0.3)
     (user_trace_width 0.2)
     (user_trace_width 0.3)
@@
       (net 2 GND))
   )
+  (dimension 15.4 (width 0.15) (layer Dwgs.User)
+    (gr_text "15.400 mm" (at -43 19.7 90) (layer Dwgs.User)
+      (effects (font (size 1 1) (thickness 0.15)))
+    )
+    (feature1 (pts (xy -39.7 12) (xy -42.286421 12)))
+    (feature2 (pts (xy -39.7 27.4) (xy -42.286421 27.4)))
+    (crossbar (pts (xy -41.7 27.4) (xy -41.7 12)))
+    (arrow1a (pts (xy -41.7 12) (xy -41.113579 13.126504)))
+    (arrow1b (pts (xy -41.7 12) (xy -42.286421 13.126504)))
+    (arrow2a (pts (xy -41.7 27.4) (xy -41.113579 26.273496)))
+    (arrow2b (pts (xy -41.7 27.4) (xy -42.286421 26.273496)))
+  )
+  (dimension 78.799998 (width 0.15) (layer Dwgs.User)
+    (gr_text "78.800 mm" (at 0 31.399999 7.271038194e-07) (layer Dwgs.User)
+      (effects (font (size 1 1) (thickness 0.15)))
+    )
+    (feature1 (pts (xy 39.399999 27.399999) (xy 39.399999 30.68642)))
+    (feature2 (pts (xy -39.399999 27.4) (xy -39.399999 30.686421)))
+    (crossbar (pts (xy -39.399999 30.1) (xy 39.399999 30.099999)))
+    (arrow1a (pts (xy 39.399999 30.099999) (xy 38.273495 30.68642)))
+    (arrow1b (pts (xy 39.399999 30.099999) (xy 38.273495 29.513578)))
+    (arrow2a (pts (xy -39.399999 30.1) (xy -38.273495 30.686421)))
+    (arrow2b (pts (xy -39.399999 30.1) (xy -38.273495 29.513579)))
+  )
+  (dimension 54.799999 (width 0.15) (layer Dwgs.User)
+    (gr_text "54.800 mm" (at -47.45 0 90) (layer Dwgs.User)
+      (effects (font (size 1 1) (thickness 0.15)))
+    )
+    (feature1 (pts (xy -39.399999 -27.399999) (xy -46.736421 -27.399999)))
+    (feature2 (pts (xy -39.399999 27.4) (xy -46.736421 27.4)))
+    (crossbar (pts (xy -46.15 27.4) (xy -46.15 -27.399999)))
+    (arrow1a (pts (xy -46.15 -27.399999) (xy -45.563579 -26.273495)))
+    (arrow1b (pts (xy -46.15 -27.399999) (xy -46.736421 -26.273495)))
+    (arrow2a (pts (xy -46.15 27.4) (xy -45.563579 26.273496)))
+    (arrow2b (pts (xy -46.15 27.4) (xy -46.736421 26.273496)))
+  )
   (gr_line (start -21.4 -10.65) (end -21.4 -4.15) (layer Edge.Cuts) (width 0.2))
   (gr_line (start -30.4 -10.65) (end -21.4 -10.65) (layer Edge.Cuts) (width 0.2))
   (gr_line (start -30.4 -4.15) (end -30.4 -10.65) (layer Edge.Cuts) (width 0.2))
   (gr_line (start -21.4 -4.15) (end -30.4 -4.15) (layer Edge.Cuts) (width 0.2))
-  (gr_line (start -3 22) (end -40 22) (layer Dwgs.User) (width 0.15))
-  (gr_line (start -3 28) (end -3 22) (layer Dwgs.User) (width 0.15))
-  (gr_line (start 3 22) (end 3 28) (layer Dwgs.User) (width 0.15))
-  (gr_line (start 3 22) (end 40 22) (layer Dwgs.User) (width 0.15))
   (gr_circle (center -37.15 14.45) (end -35.95 14.45) (layer Edge.Cuts) (width 0.2))
   (gr_circle (center -37.15 -20.449999) (end -35.95 -20.449999) (layer Edge.Cuts) (width 0.2))
@@
   (via (at -10.5 -5.5) (size 0.6) (drill 0.3) (layers F.Cu B.Cu) (net 2))
   (via (at -7.75 -14.25) (size 0.6) (drill 0.3) (layers F.Cu B.Cu) (net 2))
-  (via (at -9 -11.5) (size 0.6) (drill 0.3) (layers F.Cu B.Cu) (net 2))
   (via (at -11.25 -9.25) (size 0.6) (drill 0.3) (layers F.Cu B.Cu) (net 2))
-  (via (at -19 -14) (size 1) (drill 0.5) (layers F.Cu B.Cu) (net 2))
-  (via (at -16.25 -11.75) (size 1) (drill 0.5) (layers F.Cu B.Cu) (net 2))
   (via (at -14 -20) (size 1) (drill 0.5) (layers F.Cu B.Cu) (net 2))
   (via (at -0.25 17.5) (size 0.6) (drill 0.3) (layers F.Cu B.Cu) (net 2))
@@
   (segment (start -3.5 -13.4) (end -3.5 -13.4) (width 1) (layer B.Cu) (net 3))
   (via (at -3.5 -13.4) (size 1) (drill 0.5) (layers F.Cu B.Cu) (net 3))
+  (segment (start -19.15 -17.15) (end -22.1 -20.1) (width 1) (layer B.Cu) (net 3))
+  (segment (start -16.35 -17.15) (end -19.15 -17.15) (width 1) (layer B.Cu) (net 3))
+  (segment (start -22.975 5.175) (end -23.4 5.175) (width 0.3) (layer F.Cu) (net 3))
+  (segment (start -18.65 -11.9) (end -18.65 -11.9) (width 0.3) (layer F.Cu) (net 3))
+  (segment (start -18.65 0.85) (end -22.975 5.175) (width 0.3) (layer F.Cu) (net 3))
+  (segment (start -18.65 -11.9) (end -18.65 0.85) (width 0.3) (layer F.Cu) (net 3))
+  (via (at -18.65 -11.9) (size 0.8) (drill 0.4) (layers F.Cu B.Cu) (net 3))
+  (segment (start -18.65 -14.85) (end -16.35 -17.15) (width 0.3) (layer B.Cu) (net 3))
+  (segment (start -18.65 -11.9) (end -18.65 -14.85) (width 0.3) (layer B.Cu) (net 3))
   (segment (start 1.97499 10.19999) (end 2.775 11) (width 0.25) (layer B.Cu) (net 4))
   (segment (start -1.025 11) (end -0.22499 10.19999) (width 0.25) (layer B.Cu) (net 4))
@@
   (segment (start -2.7 -17.6) (end -2.7 -18.875) (width 0.25) (layer F.Cu) (net 4))
   (segment (start -7 -13.3) (end -2.7 -17.6) (width 0.25) (layer F.Cu) (net 4))
-  (segment (start -7 -11.15) (end -10.4 -7.6) (width 1.3) (layer F.Cu) (net 4))
+  (segment (start -7 -11.15) (end -10.4 -7.6) (width 0.5) (layer F.Cu) (net 4))
   (via (at -10.4 -7.6) (size 1) (drill 0.5) (layers F.Cu B.Cu) (net 4))
   (segment (start -10.4 -7.6) (end -11.9 -6.1) (width 0.5) (layer B.Cu) (net 4))
@@
   (via (at 21.825 10.575) (size 0.8) (drill 0.4) (layers F.Cu B.Cu) (net 4))
   (segment (start 21.825 10.575) (end 25.25 10.575) (width 0.25) (layer F.Cu) (net 4))
+  (segment (start -15.65 -11.15) (end -24.6 -20.1) (width 1) (layer F.Cu) (net 4))
+  (segment (start -7 -11.15) (end -15.65 -11.15) (width 1) (layer F.Cu) (net 4))
   (segment (start -2.375 -16.9) (end -3.1 -17.625) (width 1) (layer B.Cu) (net 5))
   (segment (start 2.9 -16.9) (end -2.375 -16.9) (width 1) (layer B.Cu) (net 5))
@@
       )
     )
+  )
+  (zone (net 0) (net_name "") (layer B.Cu) (hatch edge 0.508)
+    (connect_pads (clearance 0.508))
+    (min_thickness 0.254)
+    (keepout (tracks allowed) (vias allowed) (copperpour not_allowed))
+    (fill (arc_segments 32) (thermal_gap 0.508) (thermal_bridge_width 0.508))
+    (polygon
+      (pts
+        (xy -18.275 -14.9) (xy -20.525 -17.15) (xy -18.15 -17.15)
+      )
+    )
