File: circuit/kicad/Power.sch (KiCad schematic (older format))
At the start: 67 parts, among them J1 ILG2, J2 PA3, J3 FFC7, J4 FFC4, J5 PA2, J6 PA2, J7 FFC5, Q1 CXDM4060P, SW1 SW_DPDT_x2, SW2 220AMB16R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

Commit message: パーツ配置まではとりあえず終わらせた。後は配線すればいい。
Parts:
- removed J7: FFC5, FFC:Molex_0545480571_01x05_P0.5mm, symbol Connector_Generic:Conn_01x05
- J4: renamed from J3; footprint FFC:Molex_0545480771_01x07_P0.5mm -> Connector_PinHeader_1.00mm:PinHeader_1x12_P1.00mm_Vertical; symbol Connector_Generic:Conn_01x07 -> Connector_Generic:Conn_01x12
- R17: value 1.5k -> 1.2k
- R19: value 1.2k -> 1.5k
- renumbered J4 to J3
Connections:
- net DRV2_EN: now also J3.4 (Pin_4); no longer J3.3 (Pin_3)
- net DRV2_PN: now also J3.3 (Pin_3); no longer J3.4 (Pin_4)
- net GND: now also J1.1 (Pin_1), SW1.1 (A)
- net Rotary1: now also C7.1, J4.9 (Pin_9), RN1.1 (R1.1); no longer C10.1, J4.1 (Pin_1), RN1.4 (R4.1)
- net Rotary2: now also J4.7 (Pin_7); no longer J4.2 (Pin_2)
- net Rotary4: now also C10.1, J4.6 (Pin_6), RN1.4 (R4.1); no longer C8.1, J4.3 (Pin_3), RN1.2 (R2.1)
- net Rotary8: now also C8.1, J4.8 (Pin_8), RN1.2 (R2.1); no longer C7.1, J4.4 (Pin_4), RN1.1 (R1.1)
- net SW1: now also J4.10 (Pin_10); no longer J4.5 (Pin_5)
- net SW2: now also J4.11 (Pin_11); no longer J4.6 (Pin_6)
- net SW3: now also J4.12 (Pin_12); no longer J4.7 (Pin_7)
- net at U4.10 (OUT2): now also J6.2 (Pin_2); no longer J6.1 (Pin_1)
- net at U4.8 (OUT1): now also J6.1 (Pin_1); no longer J6.2 (Pin_2)
- net at D5.2 (BK): now also R17.1; no longer R19.1
- net at D5.4 (RK): now also R19.1; no longer R17.1
- net at R17.2: now also J4.5 (Pin_5)
- net at R18.2: now also J4.4 (Pin_4)
- net at R19.2: now also J4.3 (Pin_3)
- net at D6.1 (K): now also J4.2 (Pin_2)
- net at D7.1 (K): now also J4.1 (Pin_1)
- no-connect marks 1 -> 0
Other:
- moved on the sheet: D5, D6, D7, J3, R11, R12, R13, R17, R18, R19, R20

Commit message: hoge
Parts:
- J4: footprint Connector_PinHeader_1.00mm:PinHeader_1x12_P1.00mm_Vertical -> FFC:WürthElektronik_687112183722_01x12_P0.5mm
Other:
- note added: "100mA"
- note added: "1A"
- note added: "4.5A"
- note added: "9A"
Changed lines of the file:
@@
 F 0 "J4" V 3000 4750 50  0000 C CNN
 F 1 "FFC7" V 3000 5100 50  0000 C CNN
-F 2 "Connector_PinHeader_1.00mm:PinHeader_1x12_P1.00mm_Vertical" H 2900 5250 50  0001 C CNN
+F 2 "FFC:WürthElektronik_687112183722_01x12_P0.5mm" H 2900 5250 50  0001 C CNN
 F 3 "~" H 2900 5250 50  0001 C CNN
 	1    2900 5250
@@
 Wire Wire Line
 	9400 3250 9400 3550
+Text Notes 6950 4200 0    50   ~ 0
+4.5A
+Text Notes 10500 4200 0    50   ~ 0
+4.5A
+Text Notes 3250 950  0    50   ~ 0
+9A
+Text Notes 7500 950  0    50   ~ 0
+1A
+Text Notes 5700 950  0    50   ~ 0
+100mA
 Wire Bus Line
 	4500 3550 4500 3750

Commit message: とりあえず完成
Parts:
- SW1: footprint Switch:SSAJ120100 -> Switch:SSSS810701
Changed lines of the file:
@@
 F 0 "SW1" V 2046 1712 50  0000 R CNN
 F 1 "SW_DPDT_x2" V 1955 1712 50  0000 R CNN
-F 2 "Switch:SSAJ120100" H 2000 1900 50  0001 C CNN
+F 2 "Switch:SSSS810701" H 2000 1900 50  0001 C CNN
 F 3 "~" H 2000 1900 50  0001 C CNN
 	1    2000 1900

Commit message: 点検
Connections:
- net at U3.10 (OUT2): now also J5.2 (Pin_2); no longer J5.1 (Pin_1)
- net at U3.8 (OUT1): now also J5.1 (Pin_1); no longer J5.2 (Pin_2)
Changed lines of the file:
@@
 L Connector_Generic:Conn_01x02 J5
 U 1 1 61F9ADCD
-P 5450 6250
+P 5350 6250
 AR Path="/61F9ADCD" Ref="J5"  Part="1"
 AR Path="/61EDC519/61F9ADCD" Ref="J?"  Part="1"
 AR Path="/61F60426/61F9ADCD" Ref="J?"  Part="1"
 AR Path="/61F60BF1/61F9ADCD" Ref="J?"  Part="1"
-F 0 "J5" V 5322 6330 50  0000 L CNN
-F 1 "PA2" V 5413 6330 50  0000 L CNN
-F 2 "PA:PA_01x02" H 5450 6250 50  0001 C CNN
-F 3 "~" H 5450 6250 50  0001 C CNN
-	1    5450 6250
-	0    1    1    0
+F 0 "J5" V 5222 6330 50  0000 L CNN
+F 1 "PA2" V 5313 6330 50  0000 L CNN
+F 2 "PA:PA_01x02" H 5350 6250 50  0001 C CNN
+F 3 "~" H 5350 6250 50  0001 C CNN
+	1    5350 6250
+	0    -1   1    0
 $EndComp
 Wire Wire Line

Commit message: あとはシルクを見やすい位置にもっていくだけ。
Parts:
- D5: symbol Device:LED_ABGR -> Device:LED_ARGB
- R17: value 1.2k -> 1.5k
- R19: value 1.5k -> 1.2k
Other:
- moved on the sheet: D5
Changed lines of the file:
@@
 $EndComp
 $Comp
-L Device:LED_ABGR D5
+L Device:LED_ARGB D5
 U 1 1 61F9AEC4
 P 1650 5700
@@
 F 3 "~" H 1650 5650 50  0001 C CNN
 	1    1650 5700
-	0    1    -1   0
+	0    -1   -1   0
 $EndComp
 Wire Wire Line
 	1650 5400 1650 5500
-$Comp
-L Device:R R17
-U 1 1 61F9AECB
-P 1350 6250
-AR Path="/61F9AECB" Ref="R17"  Part="1"
-AR Path="/61EDC519/61F9AECB" Ref="R?"  Part="1"
-AR Path="/61F60426/61F9AECB" Ref="R?"  Part="1"
-AR Path="/61F60BF1/61F9AECB" Ref="R?"  Part="1"
-F 0 "R17" V 1250 6250 50  0000 C CNN
-F 1 "1.2k" V 1450 6250 50  0000 C CNN
-F 2 "Resistor_SMD:R_0603_1608Metric" V 1280 6250 50  0001 C CNN
-F 3 "~" H 1350 6250 50  0001 C CNN
-	1    1350 6250
-	1    0    0    -1
-$EndComp
 $Comp
 L Device:R R18
@@
 F 3 "~" H 1650 6250 50  0001 C CNN
 	1    1650 6250
-	1    0    0    -1
-$EndComp
-$Comp
-L Device:R R19
-U 1 1 61F9AED7
-P 1950 6250
-AR Path="/61F9AED7" Ref="R19"  Part="1"
-AR Path="/61EDC519/61F9AED7" Ref="R?"  Part="1"
-AR Path="/61F60426/61F9AED7" Ref="R?"  Part="1"
-AR Path="/61F60BF1/61F9AED7" Ref="R?"  Part="1"
-F 0 "R19" V 1850 6250 50  0000 C CNN
-F 1 "1.5k" V 2050 6250 50  0000 C CNN
-F 2 "Resistor_SMD:R_0603_1608Metric" V 1880 6250 50  0001 C CNN
-F 3 "~" H 1950 6250 50  0001 C CNN
-	1    1950 6250
 	1    0    0    -1
 $EndComp
@@
 Wire Bus Line
 	3700 3000 3700 5150
+$Comp
+L Device:R R19
+U 1 1 61F9AED7
+P 1950 6250
+AR Path="/61F9AED7" Ref="R19"  Part="1"
+AR Path="/61EDC519/61F9AED7" Ref="R?"  Part="1"
+AR Path="/61F60426/61F9AED7" Ref="R?"  Part="1"
+AR Path="/61F60BF1/61F9AED7" Ref="R?"  Part="1"
+F 0 "R19" V 1850 6250 50  0000 C CNN
+F 1 "1.2k" V 2050 6250 50  0000 C CNN
+F 2 "Resistor_SMD:R_0603_1608Metric" V 1880 6250 50  0001 C CNN
+F 3 "~" H 1950 6250 50  0001 C CNN
+	1    1950 6250
+	1    0    0    -1
+$EndComp
+$Comp
+L Device:R R17
+U 1 1 61F9AECB
+P 1350 6250
+AR Path="/61F9AECB" Ref="R17"  Part="1"
+AR Path="/61EDC519/61F9AECB" Ref="R?"  Part="1"
+AR Path="/61F60426/61F9AECB" Ref="R?"  Part="1"
+AR Path="/61F60BF1/61F9AECB" Ref="R?"  Part="1"
+F 0 "R17" V 1250 6250 50  0000 C CNN
+F 1 "1.5k" V 1450 6250 50  0000 C CNN
+F 2 "Resistor_SMD:R_0603_1608Metric" V 1280 6250 50  0001 C CNN
+F 3 "~" H 1350 6250 50  0001 C CNN
+	1    1350 6250
+	1    0    0    -1
+$EndComp
 $EndSCHEMATC
