File: circuit/kicad/Power.sch (KiCad schematic (older format))
At the start: 66 parts, among them J1 ILG2, J2 PA3, J3 FFC4, J4 FFC7, J5 PA2, J6 PA2, Q1 CXDM4060P, SW1 SW_DPDT_x2, SW2 220AMB16R, SW3 SKRPABE010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

Commit message: hoge
Parts:
- SW3, SW4, SW5: symbol SKRPABE010:Switch -> Power-rescue:Switch-SKRPABE010
- U1, U2: symbol Regulator:Regulator_GOI -> Power-rescue:Regulator_GOI-Regulator
- U3, U4: symbol DRVxxxx:DRV8874 -> Power-rescue:DRV8874-DRVxxxx
Changed lines of the file:
@@
 	4600 5650 4600 5550
 $Comp
-L DRVxxxx:DRV8874 U3
+L Power-rescue:DRV8874-DRVxxxx U3
 U 1 1 61F9ADB5
 P 5400 5350
@@
 	8000 5650 8000 5550
 $Comp
-L DRVxxxx:DRV8874 U4
+L Power-rescue:DRV8874-DRVxxxx U4
 U 1 1 61F9AE49
 P 8950 5350
@@
 $EndComp
 $Comp
-L Regulator:Regulator_GOI U1
+L Power-rescue:Regulator_GOI-Regulator U1
 U 1 1 61F9AFF7
 P 5200 1100
@@
 $EndComp
 $Comp
-L Regulator:Regulator_GOI U2
+L Power-rescue:Regulator_GOI-Regulator U2
 U 1 1 61F9B151
 P 7000 1100
@@
 	7000 1500 7500 1500
 $Comp
-L SKRPABE010:Switch SW3
+L Power-rescue:Switch-SKRPABE010 SW3
 U 1 1 61F9B19F
 P 1250 3950
@@
 $EndComp
 $Comp
-L SKRPABE010:Switch SW4
+L Power-rescue:Switch-SKRPABE010 SW4
 U 1 1 61F9B1A5
 P 2000 3950
@@
 $EndComp
 $Comp
-L SKRPABE010:Switch SW5
+L Power-rescue:Switch-SKRPABE010 SW5
 U 1 1 61F9B1AB
 P 2750 3950
