File: circuit/kicad/Power.kicad_pcb (KiCad board)
At the start: 2 copper layers, 78.8 x 54.8 mm, 66 parts, among them J1 ILG2, J2 PA3, J3 FFC4, J4 FFC7, J5 PA2, J6 PA2, Q1 CXDM4060P, SW1 SW_DPDT_x2, SW2 220AMB16R, SW3 SKRPABE010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

Commit message: Gerber データを出力した。これから先輩に添削してもらう。
Routing:
- net GND: vias 65 -> 67
