File: circuit/kicad/SubSensor.kicad_pcb (KiCad board)
At the start: 2 copper layers, 28 x 10 mm, 5 parts, among them J1 SH3, U1 S7136

Commit message: あとはシルクを見やすい位置にもっていくだけ。
Connections:
- J1 pad MP: (no net) -> GND
Changed lines of the file:
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@@
     (mod_text_size 1 1)
     (mod_text_width 0.15)
-    (pad_size 1.524 1.524)
-    (pad_drill 0.762)
+    (pad_size 1.2 1.8)
+    (pad_drill 0)
     (pad_to_mask_clearance 0)
     (aux_axis_origin 0 0)
@@
     (pad 2 smd rect (at 0 -2.525 90) (size 0.6 1.55) (layers F.Cu F.Paste F.Mask)
       (net 5 "Net-(J1-Pad2)"))
-    (pad MP smd rect (at -2.3 0 90) (size 1.2 1.8) (layers F.Cu F.Paste F.Mask))
-    (pad MP smd rect (at 2.3 0 90) (size 1.2 1.8) (layers F.Cu F.Paste F.Mask))
+    (pad MP smd rect (at -2.3 0 90) (size 1.2 1.8) (layers F.Cu F.Paste F.Mask)
+      (net 2 GND))
+    (pad MP smd rect (at 2.3 0 90) (size 1.2 1.8) (layers F.Cu F.Paste F.Mask)
+      (net 2 GND))
   )
   (module Resistor_SMD:R_0603_1608Metric (layer B.Cu)
@@
   (gr_line (start 4 8) (end 23.5 8) (layer Dwgs.User) (width 0.15))
   (gr_line (start 4 2) (end 4 8) (layer Dwgs.User) (width 0.15))
-  (segment (start 15.88 4) (end 16.15 3.73) (width 0.25) (layer B.Cu) (net 1))
+  (segment (start 15.88 4) (end 16.15 3.73) (width 0.25) (layer B.Cu) (net 1) (status 30))
   (via (at 17 5) (size 0.8) (drill 0.4) (layers F.Cu B.Cu) (net 1))
-  (segment (start 18.225 5) (end 17 5) (width 0.25) (layer F.Cu) (net 1))
+  (segment (start 18.225 5) (end 17 5) (width 0.25) (layer F.Cu) (net 1) (status 10))
   (segment (start 17 5) (end 14.5 2.5) (width 0.25) (layer B.Cu) (net 1))
   (via (at 10.5 3.5) (size 0.8) (drill 0.4) (layers F.Cu B.Cu) (net 1))
   (segment (start 11.5 2.5) (end 10.5 3.5) (width 0.25) (layer B.Cu) (net 1))
-  (segment (start 10 4) (end 5.475 4) (width 0.25) (layer F.Cu) (net 1))
+  (segment (start 10 4) (end 5.475 4) (width 0.25) (layer F.Cu) (net 1) (status 20))
   (segment (start 10.5 3.5) (end 10 4) (width 0.25) (layer F.Cu) (net 1))
   (segment (start 13 2.5) (end 13.75 2.5) (width 0.25) (layer B.Cu) (net 1))
   (segment (start 14.5 2.5) (end 13 2.5) (width 0.25) (layer B.Cu) (net 1))
   (segment (start 13 2.5) (end 11.5 2.5) (width 0.25) (layer B.Cu) (net 1))
-  (segment (start 14.325 3.075) (end 14.325 4) (width 0.25) (layer B.Cu) (net 1))
+  (segment (start 14.325 3.075) (end 14.325 4) (width 0.25) (layer B.Cu) (net 1) (status 20))
   (segment (start 13.75 2.5) (end 14.325 3.075) (width 0.25) (layer B.Cu) (net 1))
   (via (at 23 9) (size 0.8) (drill 0.4) (layers F.Cu B.Cu) (net 2))
   (via (at 23 1) (size 0.8) (drill 0.4) (layers F.Cu B.Cu) (net 2))
   (via (at 21 6.25) (size 0.8) (drill 0.4) (layers F.Cu B.Cu) (net 2))
-  (segment (start 15.88 6) (end 16.15 6.27) (width 0.25) (layer B.Cu) (net 3))
-  (segment (start 14.2875 6) (end 15.88 6) (width 0.25) (layer B.Cu) (net 3))
-  (segment (start 12.675 5.9625) (end 12.7125 6) (width 0.25) (layer B.Cu) (net 4))
-  (segment (start 12.675 4) (end 12.675 5.9625) (width 0.25) (layer B.Cu) (net 4))
-  (segment (start 5.475 5) (end 14 5) (width 0.25) (layer F.Cu) (net 5))
+  (segment (start 15.88 6) (end 16.15 6.27) (width 0.25) (layer B.Cu) (net 3) (status 30))
+  (segment (start 14.2875 6) (end 15.88 6) (width 0.25) (layer B.Cu) (net 3) (status 30))
+  (segment (start 12.675 5.9625) (end 12.7125 6) (width 0.25) (layer B.Cu) (net 4) (status 30))
+  (segment (start 12.675 4) (end 12.675 5.9625) (width 0.25) (layer B.Cu) (net 4) (status 30))
+  (segment (start 5.475 5) (end 14 5) (width 0.25) (layer F.Cu) (net 5) (status 10))
   (via (at 19 3.5) (size 0.8) (drill 0.4) (layers F.Cu B.Cu) (net 5))
   (segment (start 15.5 3.5) (end 19 3.5) (width 0.25) (layer F.Cu) (net 5))
   (segment (start 14 5) (end 15.5 3.5) (width 0.25) (layer F.Cu) (net 5))
-  (segment (start 22.62 3.5) (end 22.85 3.73) (width 0.25) (layer B.Cu) (net 5))
-  (segment (start 19 3.5) (end 22.62 3.5) (width 0.25) (layer B.Cu) (net 5))
+  (segment (start 22.62 3.5) (end 22.85 3.73) (width 0.25) (layer B.Cu) (net 5) (status 30))
+  (segment (start 19 3.5) (end 22.62 3.5) (width 0.25) (layer B.Cu) (net 5) (status 20))
   (zone (net 0) (net_name "") (layer B.Cu) (hatch edge 0.508)
     (connect_pads (clearance 0.508))
