File: circuit/kicad/FrontSensor.kicad_pcb (KiCad board)
At the start: 2 copper layers, 50 x 32.5 mm, 18 parts, among them J1 FFC6, Q1 TEMT7100X01, Q2 TEMT7100X01, Q3 TEMT7100X01, Q4 TEMT7100X01

Commit message: export
Other:
- rule via_min_size: 0.4 -> 0.6
