File: circuit/kicad/Main.kicad_pcb (KiCad board)
At the start: 2 copper layers, 110.8 x 117 mm, 104 parts, among them J1 SH3, J10 PA3, J11 SH4, J2 SH3, J3 FFC6, J4 SH6, J5 FTSH2x5, J6 FFC4, J7 SH4, J8 FFC12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

Commit message: でーきーなーいー
Connections:
- J1 pad MP: GND -> (no net)
- J11 pad MP: GND -> (no net)
- J2 pad MP: GND -> (no net)
- J3 pad MP: GND -> (no net)
- J4 pad MP: GND -> (no net)
- J6 pad 1: /DRV1_EN -> /DRV1_PN
- J6 pad 2: /DRV1_PN -> /DRV1_EN
- J6 pad 3: /DRV2_PN -> /DRV2_EN
- J6 pad 4: /DRV2_EN -> /DRV2_PN
- J6 pad MP: GND -> (no net)
- J7 pad MP: GND -> (no net)
- J8 pad MP: GND -> (no net)
- U2 pad 2: /DRV2_EN -> /DRV2_PN
- U2 pad 54: /DRV1_EN -> /DRV1_PN
- U2 pad 58: /DRV1_PN -> /DRV1_EN
- U2 pad 59: /DRV2_PN -> /DRV2_EN
- U3 pad 25: GND -> (no net)
Routing:
- net /DRV2_PN: track 35.5 -> 44.8 mm
- net /DRV2_EN: track 44.8 -> 35.5 mm
