File: circuit/kicad/SubSensor.sch (KiCad schematic (older format))
At the start: 5 parts, among them J1 SH3, U1 S7136

Commit message: testcommit
Parts:
- U1: symbol S7136:S7136 -> SubSensor-rescue:S7136-S7136
Changed lines of the file:
@@
 $Descr A4 11693 8268
 encoding utf-8
-Sheet 5 5
+Sheet 1 1
 Title ""
 Date ""
@@
 $EndDescr
 $Comp
-L S7136:S7136 U1
+L SubSensor-rescue:S7136-S7136 U1
 U 1 1 61F6138D
 P 4100 4500
